File: mk2ee_kicad_project/driver-1.sch (KiCad schematic (older format))
At the start: 33 parts, among them J12 Conn_01x03_Male, J12 Conn_01x04_Male, J3 Conn_01x02_Male, J4 Conn_01x06_Male, J5 Conn_01x06_Male, U11 TSR_1-2465, U4 NCP718xSN330, U5 DRV8818PWP, U6 74HC595

Commit message: all components are checked
Parts:
- removed C22, C23: 10uF, Capacitor_SMD:CP_Elec_6.3x5.8, symbol Device:CP1
- removed J12: Conn_01x03_Male, symbol Connector:Conn_01x03_Male
- added C17, C18: 10uF, Capacitor_SMD:CP_Elec_4x5.4, symbol Device:CP1
- added J6: Conn_01x04_Male, MK2Library:Molex_MicroClasp_55935-0430_1x04_P2.00mm_Horizontal, symbol Connector:Conn_01x04_Male
- added TP5, TP7, TP8, TP9: TestPoint, TestPoint:TestPoint_Pad_D4.0mm, symbol Connector:TestPoint
- C10, C8, C9: footprint Capacitor_SMD:C_0805_2012Metric_Pad1.15x1.40mm_HandSolder -> Capacitor_SMD:C_1206_3216Metric; Manufacturer (none) -> Kemet; Name (none) -> C1206C224K5RACTU
- C11, C12, C13: value 0.1uF -> 100nF; footprint Capacitor_SMD:C_0805_2012Metric_Pad1.15x1.40mm_HandSolder -> Capacitor_SMD:C_1206_3216Metric; Manufacturer (none) -> Kemet; Name (none) -> C1206C104K5RACTU
- C14: footprint (none) -> Capacitor_SMD:CP_Elec_6.3x7.7; Manufacturer (none) -> Panasonic; Name (none) -> EEEFK1E101XP
- C19: renamed from C17; footprint (none) -> Capacitor_SMD:C_1206_3216Metric; Manufacturer (none) -> Kemet; Name (none) -> C1206C104K5RACTU
- C6, C7: Manufacturer (none) -> MULTICOMP PRO; Name (none) -> MC1206B102K500CT
- J3: footprint Connector_Molex:Molex_CLIK-Mate_502443-0270_1x02-1MP_P2.00mm_Vertical -> MK2Library:Molex_MicroClasp_55932-0210_1x02_P2.00mm_Vertical; Name CLIK-Mate_502443-0270 -> 55932-0210
- J4, J5: value Conn_01x06_Male -> Conn_02x03_Male; footprint Connector_Molex:Molex_CLIK-Mate_502443-0670_1x06-1MP_P2.00mm_Vertical -> Connector_IDC:IDC-Header_2x03_P2.54mm_Horizontal; Manufacturer Molex -> AMPHENOL ICC; Name CLIC-Mate 502443-0670 -> T821106A1R100CEU
- J7: renamed from J12; footprint Connector_Molex:Molex_CLIK-Mate_502443-0470_1x04-1MP_P2.00mm_Vertical -> MK2Library:Molex_MicroClasp_55935-0430_1x04_P2.00mm_Horizontal; Name CLIK-Mate_502443-0470 -> 502443-0470
- R1: Manufacturer (none) -> MULTICOMP PRO; Name (none) -> MCWR12X4702FTL
- R2, R3, R4, R5: Manufacturer (none) -> MULTICOMP PRO; Name (none) -> MC0125W1206510K
- R6: footprint Resistor_SMD:R_0805_2012Metric_Pad1.15x1.40mm_HandSolder -> Resistor_SMD:R_1206_3216Metric; Manufacturer (none) -> MULTICOMP PRO; Name (none) -> MCWR12X4702FTL
- R7: value 0.2R -> 0.43R; footprint Resistor_SMD:R_0805_2012Metric_Pad1.15x1.40mm_HandSolder -> Resistor_SMD:R_1206_3216Metric; Manufacturer (none) -> BOURNS; Name (none) -> CRL1206-FW-R430ELF
- R8: value 0.2R -> 0.43R; Manufacturer (none) -> BOURNS; Name (none) -> CRL1206-FW-R430ELF
- U4: renamed from U11; Manufacturer (none) -> Traco Power; Name (none) -> TSR 2-2465
- U6: footprint (none) -> MK2Library:SN74HC595PWR; Manufacturer (none) -> Texas Instruments; Name (none) -> SN74HC595PWR
- gave numbers to parts that had none: 1
- renumbered F2 to F3, U4 to U5, U5 to U7
Connections:
- net VM2 is gone; now on net VMB: C14.1, J4.1 (Pin_1)
- net GND: now also U4.2 (GND), C17.2, C18.2, J6.2 (Pin_2)
- net PWM2: now also J6.3 (Pin_3)
- net VCC6v5: now also C18.1, J6.4 (Pin_4), TP7.1
- net VCCB3v3: now also TP9.1
- net pwr9: now reaches C15.1, F3.P$2, U5.1 (IN), U5.3 (EN)
- net pwr9: now also TP8.1
- net pwr6: now reaches F2.P$2, U4.1 (Vin)
- net pwr6: now also C17.1, TP5.1
- no-connect marks 1 -> 2
Other:
- moved on the sheet: F3

Commit message: PCB design is updated
Parts:
- C7: footprint Capacitor_SMD:C_0805_2012Metric_Pad1.15x1.40mm_HandSolder -> Capacitor_SMD:C_1206_3216Metric
Changed lines of the file:
@@
-$EndComp
-$Comp
-L Device:C C7
-U 1 1 5F478D33
-P 5700 2100
-F 0 "C7" V 5448 2100 50  0000 C CNN
-F 1 "1000pF" V 5539 2100 50  0000 C CNN
-F 2 "Capacitor_SMD:C_0805_2012Metric_Pad1.15x1.40mm_HandSolder" H 5738 1950 50  0001 C CNN
-F 3 "~" H 5700 2100 50  0001 C CNN
-F 4 "MC1206B102K500CT" V 5700 2100 50  0001 C CNN "Name"
-F 5 "MULTICOMP PRO" V 5700 2100 50  0001 C CNN "Manufacturer"
-	1    5700 2100
-	0    1    1    0
 $EndComp
 $Comp
@@
 	5850 950  5850 1300
 Wire Wire Line
-	5850 2100 5850 2450
-Wire Wire Line
 	6600 1900 5850 1900
 Wire Wire Line
@@
 Wire Wire Line
 	6600 2000 5850 2000
-Wire Wire Line
-	5850 2000 5850 2100
-Connection ~ 5850 2100
 $Comp
 L power:GND #PWR0112
@@
 Text Label 4250 6550 2    50   ~ 0
 pwr10
+Wire Wire Line
+	5850 2000 5850 2100
+$Comp
+L Device:C C7
+U 1 1 603370C1
+P 5700 2100
+F 0 "C7" V 5448 2100 50  0000 C CNN
+F 1 "1000pF" V 5539 2100 50  0000 C CNN
+F 2 "Capacitor_SMD:C_1206_3216Metric" H 5738 1950 50  0001 C CNN
+F 3 "~" H 5700 2100 50  0001 C CNN
+F 4 "MC1206B102K500CT" V 5700 2100 50  0001 C CNN "Name"
+F 5 "MULTICOMP PRO" V 5700 2100 50  0001 C CNN "Manufacturer"
+	1    5700 2100
+	0    1    1    0
+$EndComp
+Connection ~ 5850 2100
+Wire Wire Line
+	5850 2100 5850 2450
 $EndSCHEMATC

Commit message: PCB designs are updated
Parts:
- R2, R3, R4, R5: footprint Resistor_SMD:R_0805_2012Metric_Pad1.15x1.40mm_HandSolder -> Resistor_SMD:R_1206_3216Metric
Connections:
- net VCC2 is gone; now on net VCCB3v3: R2.2, R4.2
Changed lines of the file:
@@
 F 0 "R4" H 3830 2404 50  0000 R CNN
 F 1 "10k" H 3830 2495 50  0000 R CNN
-F 2 "Resistor_SMD:R_0805_2012Metric_Pad1.15x1.40mm_HandSolder" V 3830 2450 50  0001 C CNN
+F 2 "Resistor_SMD:R_1206_3216Metric" V 3830 2450 50  0001 C CNN
 F 3 "~" H 3900 2450 50  0001 C CNN
 F 4 "MC0125W1206510K" H 3900 2450 50  0001 C CNN "Name"
@@
 F 0 "R5" H 3830 2904 50  0000 R CNN
 F 1 "10k" H 3830 2995 50  0000 R CNN
-F 2 "Resistor_SMD:R_0805_2012Metric_Pad1.15x1.40mm_HandSolder" V 3830 2950 50  0001 C CNN
+F 2 "Resistor_SMD:R_1206_3216Metric" V 3830 2950 50  0001 C CNN
 F 3 "~" H 3900 2950 50  0001 C CNN
 F 4 "MC0125W1206510K" H 3900 2950 50  0001 C CNN "Name"
@@
 Connection ~ 4750 2150
 Text GLabel 3900 2100 1    50   Input ~ 0
-VCC2
+VCCB3v3
 Text GLabel 4750 1050 1    50   Input ~ 0
-VCC2
+VCCB3v3
 Text GLabel 8200 1250 1    50   Input ~ 0
 VCCB3v3
@@
 F 0 "R2" H 4680 1304 50  0000 R CNN
 F 1 "10k" H 4680 1395 50  0000 R CNN
-F 2 "Resistor_SMD:R_0805_2012Metric_Pad1.15x1.40mm_HandSolder" V 4680 1350 50  0001 C CNN
+F 2 "Resistor_SMD:R_1206_3216Metric" V 4680 1350 50  0001 C CNN
 F 3 "~" H 4750 1350 50  0001 C CNN
 F 4 "MC0125W1206510K" H 4750 1350 50  0001 C CNN "Name"
@@
 F 0 "R3" H 4680 1804 50  0000 R CNN
 F 1 "10k" H 4680 1895 50  0000 R CNN
-F 2 "Resistor_SMD:R_0805_2012Metric_Pad1.15x1.40mm_HandSolder" V 4680 1850 50  0001 C CNN
+F 2 "Resistor_SMD:R_1206_3216Metric" V 4680 1850 50  0001 C CNN
 F 3 "~" H 4750 1850 50  0001 C CNN
 F 4 "MC0125W1206510K" H 4750 1850 50  0001 C CNN "Name"

Commit message: all components are connected
Parts:
- TP5, TP7, TP8, TP9: footprint TestPoint:TestPoint_Pad_D4.0mm -> TestPoint:TestPoint_Pad_D1.5mm
Connections:
- net GND: now also J4.6 (Pin_6), J6.4 (Pin_4); no longer J4.2 (Pin_2), J6.2 (Pin_2)
- net PWM2: now also J4.4 (Pin_4), J5.4 (Pin_4), J6.2 (Pin_2); no longer J4.5 (Pin_5), J5.5 (Pin_5), J6.3 (Pin_3)
- net RESETn: now also U6.4 (QE); no longer U6.5 (QF)
- net SH-CLKDr2: now also J4.5 (Pin_5), J5.1 (Pin_1); no longer J4.6 (Pin_6), J5.6 (Pin_6)
- net SRn: now also U6.3 (QD); no longer U6.4 (QE)
- net STEP: now also U6.5 (QF); no longer U6.3 (QD)
- net SerialDataInDr2: now also J4.1 (Pin_1); no longer J4.4 (Pin_4)
- net SerialDataOutDr2: now also J5.5 (Pin_5); no longer J5.4 (Pin_4)
- net USM0: now also U6.2 (QC); no longer U6.1 (QB)
- net USM1: now also U6.1 (QB); no longer U6.2 (QC)
- net VCC6v5: now also J6.3 (Pin_3); no longer J6.4 (Pin_4)
- net VMB: now also J4.2 (Pin_2), J5.6 (Pin_6); no longer J4.1 (Pin_1), J5.1 (Pin_1)
Other:
- moved on the sheet: C14
Changed lines of the file:
@@
 L power:GND #PWR0117
 U 1 1 5F4EE14D
-P 9250 4050
-F 0 "#PWR0117" H 9250 3800 50  0001 C CNN
-F 1 "GND" H 9255 3877 50  0000 C CNN
-F 2 "" H 9250 4050 50  0001 C CNN
-F 3 "" H 9250 4050 50  0001 C CNN
-	1    9250 4050
-	0    1    1    0
-$EndComp
-Wire Wire Line
-	9250 4150 9400 4150
-Wire Wire Line
-	9250 4050 9500 4050
+P 9250 3650
+F 0 "#PWR0117" H 9250 3400 50  0001 C CNN
+F 1 "GND" H 9255 3477 50  0000 C CNN
+F 2 "" H 9250 3650 50  0001 C CNN
+F 3 "" H 9250 3650 50  0001 C CNN
+	1    9250 3650
+	-1   0    0    1
+$EndComp
 Text GLabel 2600 1850 2    50   Output ~ 0
 DIR
+Text GLabel 2600 2050 2    50   Output ~ 0
+USM0
 Text GLabel 2600 1950 2    50   Output ~ 0
-USM0
-Text GLabel 2600 2050 2    50   Output ~ 0
 USM1
+Text GLabel 2600 2350 2    50   Output ~ 0
+STEP
 Text GLabel 2600 2150 2    50   Output ~ 0
-STEP
+SRn
 Text GLabel 2600 2250 2    50   Output ~ 0
-SRn
-Text GLabel 2600 2350 2    50   Output ~ 0
 RESETn
+Text GLabel 9250 5300 0    50   Input ~ 0
+SerialDataOutDr2
 Text GLabel 9250 5400 0    50   Input ~ 0
-SerialDataOutDr2
-Text GLabel 9250 5300 0    50   Input ~ 0
 PWM2
-Text GLabel 9250 5200 0    50   Input ~ 0
+Text GLabel 9250 5700 0    50   Input ~ 0
 SH-CLKDr2
 Text GLabel 9250 5500 0    50   Input ~ 0
@@
 Text GLabel 1300 1850 0    50   Input ~ 0
 SerialDataInDr2
-Text GLabel 9250 5700 0    50   Input ~ 0
+Text GLabel 9250 5200 0    50   Input ~ 0
 VMB
 $Comp
@@
 Text GLabel 9250 3950 0    50   Output ~ 0
 PO-CLKDr2
-Text GLabel 9250 3650 0    50   Output ~ 0
+Text GLabel 9250 3750 0    50   Output ~ 0
 SH-CLKDr2
-Text GLabel 9250 3750 0    50   Output ~ 0
+Text GLabel 9250 3850 0    50   Output ~ 0
 PWM2
-Text GLabel 9250 3850 0    50   Output ~ 0
+Text GLabel 9250 4150 0    50   Output ~ 0
 SerialDataInDr2
 $Comp
@@
 Wire Wire Line
 	9250 2950 9500 2950
-Text GLabel 9250 4150 0    50   Output ~ 0
+Text GLabel 8300 4050 0    50   Output ~ 0
 VMB
-Wire Wire Line
-	9400 4300 9400 4150
-Connection ~ 9400 4150
-Wire Wire Line
-	9400 4150 9500 4150
 $Comp
 L power:GND #PWR0137
 U 1 1 5F975427
-P 9400 4600
-F 0 "#PWR0137" H 9400 4350 50  0001 C CNN
-F 1 "GND" H 9405 4427 50  0000 C CNN
-F 2 "" H 9400 4600 50  0001 C CNN
-F 3 "" H 9400 4600 50  0001 C CNN
-	1    9400 4600
+P 8500 4500
+F 0 "#PWR0137" H 8500 4250 50  0001 C CNN
+F 1 "GND" H 8505 4327 50  0000 C CNN
+F 2 "" H 8500 4500 50  0001 C CNN
+F 3 "" H 8500 4500 50  0001 C CNN
+	1    8500 4500
 	1    0    0    -1
 $EndComp
@@
 L power:GND #PWR0145
 U 1 1 5FC7793A
-P 9350 6250
-F 0 "#PWR0145" H 9350 6000 50  0001 C CNN
-F 1 "GND" H 9355 6077 50  0000 C CNN
-F 2 "" H 9350 6250 50  0001 C CNN
-F 3 "" H 9350 6250 50  0001 C CNN
-	1    9350 6250
-	1    0    0    -1
-$EndComp
-Text GLabel 9000 5950 0    50   Input ~ 0
+P 8850 5950
+F 0 "#PWR0145" H 8850 5700 50  0001 C CNN
+F 1 "GND" H 8855 5777 50  0000 C CNN
+F 2 "" H 8850 5950 50  0001 C CNN
+F 3 "" H 8850 5950 50  0001 C CNN
+	1    8850 5950
+	1    0    0    -1
+$EndComp
+Text GLabel 9300 6050 0    50   Input ~ 0
 VCC6v5
 Wire Wire Line
-	9000 5950 9500 5950
-Wire Wire Line
 	9350 6250 9350 6150
 Wire Wire Line
 	9350 6150 9500 6150
-Text GLabel 9300 6050 0    50   Input ~ 0
+Text GLabel 9350 6250 0    50   Input ~ 0
 PWM2
 Wire Wire Line
@@
 L Device:CP1 C?
 U 1 1 602E4B0B
-P 9400 4450
+P 8500 4350
 AR Path="/5F455032/602E4B0B" Ref="C?"  Part="1"
 AR Path="/5F4C637B/602E4B0B" Ref="C?"  Part="1"
 AR Path="/5F475AB3/602E4B0B" Ref="C14"  Part="1"
-F 0 "C14" H 9515 4496 50  0000 L CNN
-F 1 "100uF" H 9515 4405 50  0000 L CNN
-F 2 "Capacitor_SMD:CP_Elec_6.3x7.7" H 9400 4450 50  0001 C CNN
-F 3 "~" H 9400 4450 50  0001 C CNN
-F 4 "EEEFK1E101XP" H 9400 4450 50  0001 C CNN "Name"
-F 5 "Panasonic" H 9400 4450 50  0001 C CNN "Manufacturer"
-	1    9400 4450
+F 0 "C14" H 8615 4396 50  0000 L CNN
+F 1 "100uF" H 8615 4305 50  0000 L CNN
+F 2 "Capacitor_SMD:CP_Elec_6.3x7.7" H 8500 4350 50  0001 C CNN
+F 3 "~" H 8500 4350 50  0001 C CNN
+F 4 "EEEFK1E101XP" H 8500 4350 50  0001 C CNN "Name"
+F 5 "Panasonic" H 8500 4350 50  0001 C CNN "Manufacturer"
+	1    8500 4350
 	1    0    0    -1
 $EndComp
@@
 F 0 "TP5" H 2358 5068 50  0000 L CNN
 F 1 "TestPoint" H 2358 4977 50  0001 L CNN
-F 2 "TestPoint:TestPoint_Pad_D4.0mm" H 2500 4950 50  0001 C CNN
+F 2 "TestPoint:TestPoint_Pad_D1.5mm" H 2500 4950 50  0001 C CNN
 F 3 "~" H 2500 4950 50  0001 C CNN
 	1    2300 4950
@@
 F 0 "TP7" H 3908 5068 50  0000 L CNN
 F 1 "TestPoint" H 3908 4977 50  0001 L CNN
-F 2 "TestPoint:TestPoint_Pad_D4.0mm" H 4050 4950 50  0001 C CNN
+F 2 "TestPoint:TestPoint_Pad_D1.5mm" H 4050 4950 50  0001 C CNN
 F 3 "~" H 4050 4950 50  0001 C CNN
 	1    3850 4950
@@
 F 0 "TP8" H 2508 6468 50  0000 L CNN
 F 1 "TestPoint" H 2508 6377 50  0001 L CNN
-F 2 "TestPoint:TestPoint_Pad_D4.0mm" H 2650 6350 50  0001 C CNN
+F 2 "TestPoint:TestPoint_Pad_D1.5mm" H 2650 6350 50  0001 C CNN
 F 3 "~" H 2650 6350 50  0001 C CNN
 	1    2450 6350
@@
 F 0 "TP9" H 3858 6468 50  0000 L CNN
 F 1 "TestPoint" H 3858 6377 50  0001 L CNN
-F 2 "TestPoint:TestPoint_Pad_D4.0mm" H 4000 6350 50  0001 C CNN
+F 2 "TestPoint:TestPoint_Pad_D1.5mm" H 4000 6350 50  0001 C CNN
 F 3 "~" H 4000 6350 50  0001 C CNN
 	1    3800 6350
@@
 Wire Wire Line
 	5850 2100 5850 2450
+Wire Wire Line
+	8850 5950 9500 5950
+Wire Wire Line
+	9250 4150 9500 4150
+Wire Wire Line
+	8300 4050 8500 4050
+Wire Wire Line
+	8500 4200 8500 4050
+Connection ~ 8500 4050
+Wire Wire Line
+	8500 4050 9500 4050
 $EndSCHEMATC

Commit message: New 3D model of Base part and PCB design is fixed
Parts:
- added TP11: TestPoint, TestPoint:TestPoint_THTPad_D1.0mm_Drill0.5mm, symbol Connector:TestPoint
- C10, C11, C12, C13, C15, C16, C19, C6, C7, C8, C9: footprint Capacitor_SMD:C_1206_3216Metric -> Capacitor_SMD:C_1206_3216Metric_Pad1.42x1.75mm_HandSolder
- R1, R2, R3, R4, R5, R6, R7: footprint Resistor_SMD:R_1206_3216Metric -> Resistor_SMD:R_1206_3216Metric_Pad1.42x1.75mm_HandSolder
- R8: footprint Resistor_SMD:R_0805_2012Metric_Pad1.15x1.40mm_HandSolder -> Resistor_SMD:R_1206_3216Metric_Pad1.42x1.75mm_HandSolder
- TP5, TP7, TP8, TP9: footprint TestPoint:TestPoint_Pad_D1.5mm -> TestPoint:TestPoint_THTPad_D1.0mm_Drill0.5mm
- U5: footprint Package_TO_SOT_SMD:SOT-23-5 -> Package_TO_SOT_SMD:SOT-23-5_HandSoldering
Connections:
- net GND: now also TP11.1
Changed lines of the file:
@@
 F 0 "R7" V 4243 3200 50  0000 C CNN
 F 1 "0.43R" V 4334 3200 50  0000 C CNN
-F 2 "Resistor_SMD:R_1206_3216Metric" V 4380 3200 50  0001 C CNN
+F 2 "Resistor_SMD:R_1206_3216Metric_Pad1.42x1.75mm_HandSolder" V 4380 3200 50  0001 C CNN
 F 3 "~" H 4450 3200 50  0001 C CNN
 F 4 "CRL1206-FW-R430ELF " V 4450 3200 50  0001 C CNN "Name"
@@
 F 0 "C6" V 5448 950 50  0000 C CNN
 F 1 "1000pF" V 5539 950 50  0000 C CNN
-F 2 "Capacitor_SMD:C_1206_3216Metric" H 5738 800 50  0001 C CNN
+F 2 "Capacitor_SMD:C_1206_3216Metric_Pad1.42x1.75mm_HandSolder" H 5738 800 50  0001 C CNN
 F 3 "~" H 5700 950 50  0001 C CNN
 F 4 "MC1206B102K500CT" V 5700 950 50  0001 C CNN "Name"
@@
 F 0 "R1" V 5493 1300 50  0000 C CNN
 F 1 "47k" V 5584 1300 50  0000 C CNN
-F 2 "Resistor_SMD:R_1206_3216Metric" V 5630 1300 50  0001 C CNN
+F 2 "Resistor_SMD:R_1206_3216Metric_Pad1.42x1.75mm_HandSolder" V 5630 1300 50  0001 C CNN
 F 3 "~" H 5700 1300 50  0001 C CNN
 F 4 "MCWR12X4702FTL" V 5700 1300 50  0001 C CNN "Name"
@@
 F 0 "R6" V 5493 2450 50  0000 C CNN
 F 1 "47k" V 5584 2450 50  0000 C CNN
-F 2 "Resistor_SMD:R_1206_3216Metric" V 5630 2450 50  0001 C CNN
+F 2 "Resistor_SMD:R_1206_3216Metric_Pad1.42x1.75mm_HandSolder" V 5630 2450 50  0001 C CNN
 F 3 "~" H 5700 2450 50  0001 C CNN
 F 4 "MCWR12X4702FTL" V 5700 2450 50  0001 C CNN "Name"
@@
 F 0 "R8" V 4243 3550 50  0000 C CNN
 F 1 "0.43R" V 4334 3550 50  0000 C CNN
-F 2 "Resistor_SMD:R_0805_2012Metric_Pad1.15x1.40mm_HandSolder" V 4380 3550 50  0001 C CNN
+F 2 "Resistor_SMD:R_1206_3216Metric_Pad1.42x1.75mm_HandSolder" V 4380 3550 50  0001 C CNN
 F 3 "~" H 4450 3550 50  0001 C CNN
 F 4 "CRL1206-FW-R430ELF " V 4450 3550 50  0001 C CNN "Name"
@@
 F 0 "R4" H 3830 2404 50  0000 R CNN
 F 1 "10k" H 3830 2495 50  0000 R CNN
-F 2 "Resistor_SMD:R_1206_3216Metric" V 3830 2450 50  0001 C CNN
+F 2 "Resistor_SMD:R_1206_3216Metric_Pad1.42x1.75mm_HandSolder" V 3830 2450 50  0001 C CNN
 F 3 "~" H 3900 2450 50  0001 C CNN
 F 4 "MC0125W1206510K" H 3900 2450 50  0001 C CNN "Name"
@@
 F 0 "R5" H 3830 2904 50  0000 R CNN
 F 1 "10k" H 3830 2995 50  0000 R CNN
-F 2 "Resistor_SMD:R_1206_3216Metric" V 3830 2950 50  0001 C CNN
+F 2 "Resistor_SMD:R_1206_3216Metric_Pad1.42x1.75mm_HandSolder" V 3830 2950 50  0001 C CNN
 F 3 "~" H 3900 2950 50  0001 C CNN
 F 4 "MC0125W1206510K" H 3900 2950 50  0001 C CNN "Name"
@@
 F 0 "C8" H 6265 2996 50  0000 L CNN
 F 1 "0.22uF" H 6265 2905 50  0000 L CNN
-F 2 "Capacitor_SMD:C_1206_3216Metric" H 6188 2800 50  0001 C CNN
+F 2 "Capacitor_SMD:C_1206_3216Metric_Pad1.42x1.75mm_HandSolder" H 6188 2800 50  0001 C CNN
 F 3 "~" H 6150 2950 50  0001 C CNN
 F 4 "C1206C224K5RACTU" H 6150 2950 50  0001 C CNN "Name"
@@
 F 0 "C15" H 2415 6846 50  0000 L CNN
 F 1 "1uF" H 2415 6755 50  0000 L CNN
-F 2 "Capacitor_SMD:C_1206_3216Metric" H 2338 6650 50  0001 C CNN
+F 2 "Capacitor_SMD:C_1206_3216Metric_Pad1.42x1.75mm_HandSolder" H 2338 6650 50  0001 C CNN
 F 3 "~" H 2300 6800 50  0001 C CNN
 	1    2300 6800
@@
 F 0 "C16" H 4165 6946 50  0000 L CNN
 F 1 "1uF" H 4165 6855 50  0000 L CNN
-F 2 "Capacitor_SMD:C_1206_3216Metric" H 4088 6750 50  0001 C CNN
+F 2 "Capacitor_SMD:C_1206_3216Metric_Pad1.42x1.75mm_HandSolder" H 4088 6750 50  0001 C CNN
 F 3 "~" H 4050 6900 50  0001 C CNN
 	1    4050 6900
@@
 F 0 "U5" H 3200 7017 50  0000 C CNN
 F 1 "NCP718xSN330" H 3200 6926 50  0000 C CNN
-F 2 "Package_TO_SOT_SMD:SOT-23-5" H 3200 7000 50  0001 C CNN
+F 2 "Package_TO_SOT_SMD:SOT-23-5_HandSoldering" H 3200 7000 50  0001 C CNN
 F 3 "https://www.onsemi.com/pub/Collateral/NCP718-D.PDF" H 3200 7150 50  0001 C CNN
 	1    3200 6650
@@
 F 0 "C19" H 1215 1446 50  0000 L CNN
 F 1 "100nF" H 1215 1355 50  0000 L CNN
-F 2 "Capacitor_SMD:C_1206_3216Metric" H 1138 1250 50  0001 C CNN
+F 2 "Capacitor_SMD:C_1206_3216Metric_Pad1.42x1.75mm_HandSolder" H 1138 1250 50  0001 C CNN
 F 3 "~" H 1100 1400 50  0001 C CNN
 F 4 "C1206C104K5RACTU" H 1100 1400 50  0001 C CNN "Name"
@@
 F 0 "C13" H 4415 1896 50  0000 L CNN
 F 1 "100nF" H 4415 1805 50  0000 L CNN
-F 2 "Capacitor_SMD:C_1206_3216Metric" H 4338 1700 50  0001 C CNN
+F 2 "Capacitor_SMD:C_1206_3216Metric_Pad1.42x1.75mm_HandSolder" H 4338 1700 50  0001 C CNN
 F 3 "~" H 4300 1850 50  0001 C CNN
 F 4 "C1206C104K5RACTU" H 4300 1850 50  0001 C CNN "Name"
@@
 F 0 "C11" H 6015 4496 50  0000 L CNN
 F 1 "100nF" H 6015 4405 50  0000 L CNN
-F 2 "Capacitor_SMD:C_1206_3216Metric" H 5938 4300 50  0001 C CNN
+F 2 "Capacitor_SMD:C_1206_3216Metric_Pad1.42x1.75mm_HandSolder" H 5938 4300 50  0001 C CNN
 F 3 "~" H 5900 4450 50  0001 C CNN
 F 4 "C1206C104K5RACTU" H 5900 4450 50  0001 C CNN "Name"
@@
 F 0 "C12" H 6465 4496 50  0000 L CNN
 F 1 "100nF" H 6465 4405 50  0000 L CNN
-F 2 "Capacitor_SMD:C_1206_3216Metric" H 6388 4300 50  0001 C CNN
+F 2 "Capacitor_SMD:C_1206_3216Metric_Pad1.42x1.75mm_HandSolder" H 6388 4300 50  0001 C CNN
 F 3 "~" H 6350 4450 50  0001 C CNN
 F 4 "C1206C104K5RACTU" H 6350 4450 50  0001 C CNN "Name"
@@
 F 0 "C9" H 4965 4496 50  0000 L CNN
 F 1 "0.22uF" H 4965 4405 50  0000 L CNN
-F 2 "Capacitor_SMD:C_1206_3216Metric" H 4888 4300 50  0001 C CNN
+F 2 "Capacitor_SMD:C_1206_3216Metric_Pad1.42x1.75mm_HandSolder" H 4888 4300 50  0001 C CNN
 F 3 "~" H 4850 4450 50  0001 C CNN
 F 4 "C1206C224K5RACTU" H 4850 4450 50  0001 C CNN "Name"
@@
 F 0 "C10" H 5465 4496 50  0000 L CNN
 F 1 "0.22uF" H 5465 4405 50  0000 L CNN
-F 2 "Capacitor_SMD:C_1206_3216Metric" H 5388 4300 50  0001 C CNN
+F 2 "Capacitor_SMD:C_1206_3216Metric_Pad1.42x1.75mm_HandSolder" H 5388 4300 50  0001 C CNN
 F 3 "~" H 5350 4450 50  0001 C CNN
 F 4 "C1206C224K5RACTU" H 5350 4450 50  0001 C CNN "Name"
@@
 F 0 "R2" H 4680 1304 50  0000 R CNN
 F 1 "10k" H 4680 1395 50  0000 R CNN
-F 2 "Resistor_SMD:R_1206_3216Metric" V 4680 1350 50  0001 C CNN
+F 2 "Resistor_SMD:R_1206_3216Metric_Pad1.42x1.75mm_HandSolder" V 4680 1350 50  0001 C CNN
 F 3 "~" H 4750 1350 50  0001 C CNN
 F 4 "MC0125W1206510K" H 4750 1350 50  0001 C CNN "Name"
@@
 F 0 "R3" H 4680 1804 50  0000 R CNN
 F 1 "10k" H 4680 1895 50  0000 R CNN
-F 2 "Resistor_SMD:R_1206_3216Metric" V 4680 1850 50  0001 C CNN
+F 2 "Resistor_SMD:R_1206_3216Metric_Pad1.42x1.75mm_HandSolder" V 4680 1850 50  0001 C CNN
 F 3 "~" H 4750 1850 50  0001 C CNN
 F 4 "MC0125W1206510K" H 4750 1850 50  0001 C CNN "Name"
@@
 F 0 "TP5" H 2358 5068 50  0000 L CNN
 F 1 "TestPoint" H 2358 4977 50  0001 L CNN
-F 2 "TestPoint:TestPoint_Pad_D1.5mm" H 2500 4950 50  0001 C CNN
+F 2 "TestPoint:TestPoint_THTPad_D1.0mm_Drill0.5mm" H 2500 4950 50  0001 C CNN
 F 3 "~" H 2500 4950 50  0001 C CNN
 	1    2300 4950
@@
 F 0 "TP7" H 3908 5068 50  0000 L CNN
 F 1 "TestPoint" H 3908 4977 50  0001 L CNN
-F 2 "TestPoint:TestPoint_Pad_D1.5mm" H 4050 4950 50  0001 C CNN
+F 2 "TestPoint:TestPoint_THTPad_D1.0mm_Drill0.5mm" H 4050 4950 50  0001 C CNN
 F 3 "~" H 4050 4950 50  0001 C CNN
 	1    3850 4950
@@
 F 0 "TP8" H 2508 6468 50  0000 L CNN
 F 1 "TestPoint" H 2508 6377 50  0001 L CNN
-F 2 "TestPoint:TestPoint_Pad_D1.5mm" H 2650 6350 50  0001 C CNN
+F 2 "TestPoint:TestPoint_THTPad_D1.0mm_Drill0.5mm" H 2650 6350 50  0001 C CNN
 F 3 "~" H 2650 6350 50  0001 C CNN
 	1    2450 6350
@@
 F 0 "TP9" H 3858 6468 50  0000 L CNN
 F 1 "TestPoint" H 3858 6377 50  0001 L CNN
-F 2 "TestPoint:TestPoint_Pad_D1.5mm" H 4000 6350 50  0001 C CNN
+F 2 "TestPoint:TestPoint_THTPad_D1.0mm_Drill0.5mm" H 4000 6350 50  0001 C CNN
 F 3 "~" H 4000 6350 50  0001 C CNN
 	1    3800 6350
@@
 F 0 "C7" V 5448 2100 50  0000 C CNN
 F 1 "1000pF" V 5539 2100 50  0000 C CNN
-F 2 "Capacitor_SMD:C_1206_3216Metric" H 5738 1950 50  0001 C CNN
+F 2 "Capacitor_SMD:C_1206_3216Metric_Pad1.42x1.75mm_HandSolder" H 5738 1950 50  0001 C CNN
 F 3 "~" H 5700 2100 50  0001 C CNN
 F 4 "MC1206B102K500CT" V 5700 2100 50  0001 C CNN "Name"
@@
 Wire Wire Line
 	8500 4050 9500 4050
+$Comp
+L Connector:TestPoint TP?
+U 1 1 608D59EB
+P 2050 3750
+AR Path="/5F455032/608D59EB" Ref="TP?"  Part="1"
+AR Path="/5F4C637B/608D59EB" Ref="TP?"  Part="1"
+AR Path="/5F475AB3/608D59EB" Ref="TP11"  Part="1"
+F 0 "TP11" H 2108 3868 50  0000 L CNN
+F 1 "TestPoint" H 2108 3777 50  0001 L CNN
+F 2 "TestPoint:TestPoint_THTPad_D1.0mm_Drill0.5mm" H 2250 3750 50  0001 C CNN
+F 3 "~" H 2250 3750 50  0001 C CNN
+	1    2050 3750
+	1    0    0    -1
+$EndComp
+$Comp
+L power:GND #PWR?
+U 1 1 608D78DE
+P 2050 3750
+AR Path="/5F4C6CE4/608D78DE" Ref="#PWR?"  Part="1"
+AR Path="/5F4C6BF4/608D78DE" Ref="#PWR?"  Part="1"
+AR Path="/5F475AB3/608D78DE" Ref="#PWR?"  Part="1"
+F 0 "#PWR?" H 2050 3500 50  0001 C CNN
+F 1 "GND" H 2055 3577 50  0000 C CNN
+F 2 "" H 2050 3750 50  0001 C CNN
+F 3 "" H 2050 3750 50  0001 C CNN
+	1    2050 3750
+	1    0    0    -1
+$EndComp
 $EndSCHEMATC
