File: mk2ee_kicad_project/encoder-2.sch (KiCad schematic (older format))
At the start: 7 parts, among them J10 Conn_01x05_Male, J11 Conn_01x06_Male, J9 Conn_01x12_Male, U10 AS5047D-ATSM, U9 74HC595

Commit message: all components are checked
Parts:
- removed J10: Conn_01x05_Male, Connector_Molex:Molex_CLIK-Mate_502386-0570_1x05-1MP_P1.25mm_Horizontal, symbol Connector:Conn_01x05_Male
- removed J11: Conn_01x06_Male, Connector_Molex:Molex_CLIK-Mate_502443-0670_1x06-1MP_P2.00mm_Vertical, symbol Connector:Conn_01x06_Male
- removed J9: Conn_01x12_Male, Connector_Molex:Molex_CLIK-Mate_502443-1270_1x12-1MP_P2.00mm_Vertical, symbol Connector:Conn_01x12_Male
- removed U9: 74HC595, symbol 74xx:74HC595
- added J11: Conn_02x6_Male, Connector_PinSocket_2.54mm:PinSocket_2x06_P2.54mm_Horizontal, symbol Connector:Conn_01x12_Male
- added J12, J13: Conn_02x03_Male, MK2Library:901303206, symbol Connector:Conn_01x06_Male
- added U11: 74HC595, MK2Library:SN74HC595PWR, symbol 74xx:74HC595
- renumbered C20 to C22, C21 to C23
Connections:
- net CLKEn4: now also J11.5 (Pin_5), J12.3 (Pin_3)
- net CSn4: now also U11.15 (QA)
- net GND: now also J11.2 (Pin_2), J13.1 (Pin_1), U11.13 (~OE), U11.8 (GND)
- net MISO4: now also J11.6 (Pin_6), J12.4 (Pin_4)
- net PO-CLKDr4: now also J11.11 (Pin_11), J13.4 (Pin_4)
- net PO-CLKEn4: now also J11.8 (Pin_8), J12.1 (Pin_1), U11.12 (RCLK)
- net PWM4: now also J11.4 (Pin_4), J13.6 (Pin_6)
- net SH-CLKDr4: now also J11.12 (Pin_12), J13.5 (Pin_5)
- net SH-CLKEn4: now also J11.9 (Pin_9), J12.5 (Pin_5), U11.11 (SRCLK)
- net SerialDataInEn4: now also J11.7 (Pin_7), U11.14 (SER)
- net SerialDataOutEn4: now also J12.2 (Pin_2), U11.9 (QH')
- net VCCF3v3: now also J11.3 (Pin_3), U11.10 (~SRCLR), U11.16 (VCC)
- net VMC: now also J11.1 (Pin_1), J13.2 (Pin_2)
- new net SerialDataDr4: J11.10 (Pin_10), J13.3 (Pin_3)
- no-connect marks 14 -> 15
Changed lines of the file:
@@
 Sheet 5 5
 Title "Encoder2 - PCB4"
-Date "2020-09-03"
+Date "2021-02-09"
 Rev "1"
 Comp "ETSETB/UPC"
@@
 	9650 2850 9900 2850
 Wire Wire Line
-	9650 2950 9900 2950
+	9650 2950 9850 2950
 Text GLabel 9650 2750 0    50   Output ~ 0
 CLKEn4
@@
 	1    0    0    -1
 $EndComp
-$Comp
-L Connector:Conn_01x12_Male J9
-U 1 1 5F50E8F5
-P 10100 2650
-F 0 "J9" H 10072 2487 50  0000 R CNN
-F 1 "Conn_01x12_Male" H 10072 2578 50  0000 R CNN
-F 2 "Connector_Molex:Molex_CLIK-Mate_502443-1270_1x12-1MP_P2.00mm_Vertical" H 10100 2650 50  0001 C CNN
-F 3 "~" H 10100 2650 50  0001 C CNN
-F 4 "CLIK-Mate 502443-1207" H 10072 2669 50  0000 R CNN "Name"
-F 5 "Molex" H 10100 2650 50  0001 C CNN "Manufacturer"
-	1    10100 2650
-	-1   0    0    1
-$EndComp
 Text GLabel 9650 2150 0    50   Output ~ 0
 PO-CLKDr4
@@
 VCCF3v3
 Text GLabel 9650 2250 0    50   Output ~ 0
-SerialDataInDr4
+SerialDataDr4
 Text GLabel 9650 3150 0    50   Output ~ 0
 VMC
@@
 	9650 3150 9900 3150
 Wire Wire Line
-	9650 3700 9900 3700
-Wire Wire Line
-	9650 3800 9900 3800
-Wire Wire Line
-	9650 3900 9900 3900
-Wire Wire Line
-	9650 4000 9900 4000
-Wire Wire Line
-	9650 4100 9900 4100
-Text GLabel 9650 3900 0    50   Input ~ 0
+	9650 3850 9900 3850
+Wire Wire Line
+	9650 3950 9900 3950
+Wire Wire Line
+	9650 4050 9900 4050
+Wire Wire Line
+	9650 4150 9900 4150
+Wire Wire Line
+	9650 4250 9900 4250
+Text GLabel 9650 4050 0    50   Input ~ 0
 CLKEn4
-Text GLabel 9650 3800 0    50   Input ~ 0
+Text GLabel 9650 3950 0    50   Input ~ 0
 MISO4
-Text GLabel 9650 3700 0    50   Input ~ 0
+Text GLabel 9650 3850 0    50   Input ~ 0
 SH-CLKEn4
-Text GLabel 9650 4000 0    50   Input ~ 0
+Text GLabel 9650 4150 0    50   Input ~ 0
 SerialDataOutEn4
-Text GLabel 9650 4100 0    50   Input ~ 0
+Text GLabel 9650 4250 0    50   Input ~ 0
 PO-CLKEn4
-Text GLabel 9550 4900 0    50   Input ~ 0
-SerialDataOutDr4
-Text GLabel 9550 4700 0    50   Input ~ 0
+Text GLabel 9550 5050 0    50   Input ~ 0
+SerialDataDr4
+Text GLabel 9550 4850 0    50   Input ~ 0
 SH-CLKDr4
-Text GLabel 9550 4800 0    50   Input ~ 0
+Text GLabel 9550 4950 0    50   Input ~ 0
 PO-CLKDr4
-Text GLabel 9550 5000 0    50   Input ~ 0
+Text GLabel 9550 5150 0    50   Input ~ 0
 VMC
 Wire Wire Line
-	9550 4700 9900 4700
-Wire Wire Line
-	9550 4800 9900 4800
-Wire Wire Line
-	9550 4900 9900 4900
-Wire Wire Line
-	9550 5000 9900 5000
-Wire Wire Line
-	9900 5100 9150 5100
-Wire Wire Line
-	9150 5100 9150 5250
+	9550 4850 9900 4850
+Wire Wire Line
+	9550 4950 9900 4950
+Wire Wire Line
+	9550 5050 9900 5050
+Wire Wire Line
+	9550 5150 9900 5150
+Wire Wire Line
+	9900 5250 9150 5250
+Wire Wire Line
+	9150 5250 9150 5400
 $Comp
 L power:GND #PWR?
 U 1 1 5F53EADC
-P 9150 5250
+P 9150 5400
 AR Path="/5F4C6CE4/5F53EADC" Ref="#PWR?"  Part="1"
 AR Path="/5F4C6BF4/5F53EADC" Ref="#PWR?"  Part="1"
 AR Path="/5F505E68/5F53EADC" Ref="#PWR0134"  Part="1"
-F 0 "#PWR0134" H 9150 5000 50  0001 C CNN
-F 1 "GND" H 9155 5077 50  0000 C CNN
-F 2 "" H 9150 5250 50  0001 C CNN
-F 3 "" H 9150 5250 50  0001 C CNN
-	1    9150 5250
-	1    0    0    -1
-$EndComp
-$Comp
-L Connector:Conn_01x05_Male J10
-U 1 1 5F5D61FE
-P 10100 3900
-F 0 "J10" H 10072 3787 50  0000 R CNN
-F 1 "Conn_01x05_Male" H 10072 3878 50  0000 R CNN
-F 2 "Connector_Molex:Molex_CLIK-Mate_502386-0570_1x05-1MP_P1.25mm_Horizontal" H 10100 3900 50  0001 C CNN
-F 3 "~" H 10100 3900 50  0001 C CNN
-F 4 "CLIK-Mate_502386-0570" H 10072 3969 50  0000 R CNN "Name"
-F 5 "Molex" H 10100 3900 50  0001 C CNN "Manufacturer"
-	1    10100 3900
-	-1   0    0    1
+F 0 "#PWR0134" H 9150 5150 50  0001 C CNN
+F 1 "GND" H 9155 5227 50  0000 C CNN
+F 2 "" H 9150 5400 50  0001 C CNN
+F 3 "" H 9150 5400 50  0001 C CNN
+	1    9150 5400
+	1    0    0    -1
 $EndComp
 $Comp
@@
 Wire Wire Line
 	3850 3200 4100 3200
-$Comp
-L 74xx:74HC595 U?
-U 1 1 5F9DF230
-P 3450 3000
-AR Path="/5F4C6CE4/5F9DF230" Ref="U?"  Part="1"
-AR Path="/5F505E68/5F9DF230" Ref="U9"  Part="1"
-F 0 "U9" H 3450 3781 50  0000 C CNN
-F 1 "74HC595" H 3450 3690 50  0000 C CNN
-F 2 "" H 3450 3000 50  0001 C CNN
-F 3 "http://www.ti.com/lit/ds/symlink/sn74hc595.pdf" H 3450 3000 50  0001 C CNN
-	1    3450 3000
-	1    0    0    -1
-$EndComp
 Wire Wire Line
 	3450 2000 3450 2400
@@
 AR Path="/5F4C6CE4/5F9DF237" Ref="#PWR?"  Part="1"
 AR Path="/5F4C6BF4/5F9DF237" Ref="#PWR?"  Part="1"
-AR Path="/5F505E68/5F9DF237" Ref="#PWR?"  Part="1"
-F 0 "#PWR?" H 3450 3450 50  0001 C CNN
+AR Path="/5F505E68/5F9DF237" Ref="#PWR0149"  Part="1"
+F 0 "#PWR0149" H 3450 3450 50  0001 C CNN
 F 1 "GND" H 3455 3527 50  0000 C CNN
 F 2 "" H 3450 3700 50  0001 C CNN
@@
 Wire Wire Line
 	2950 3700 3450 3700
-Connection ~ 3450 3700
 Wire Wire Line
 	3050 2900 2900 2900
@@
 P 2600 2150
 AR Path="/5F4C6CE4/5F9DF246" Ref="C?"  Part="1"
-AR Path="/5F505E68/5F9DF246" Ref="C20"  Part="1"
-F 0 "C20" H 2715 2196 50  0000 L CNN
+AR Path="/5F505E68/5F9DF246" Ref="C22"  Part="1"
+F 0 "C22" H 2715 2196 50  0000 L CNN
 F 1 "100nF" H 2715 2105 50  0000 L CNN
 F 2 "" H 2638 2000 50  0001 C CNN
@@
 AR Path="/5F4C6CE4/5F9DF24E" Ref="#PWR?"  Part="1"
 AR Path="/5F4C6BF4/5F9DF24E" Ref="#PWR?"  Part="1"
-AR Path="/5F505E68/5F9DF24E" Ref="#PWR?"  Part="1"
-F 0 "#PWR?" H 2600 2050 50  0001 C CNN
+AR Path="/5F505E68/5F9DF24E" Ref="#PWR0150"  Part="1"
+F 0 "#PWR0150" H 2600 2050 50  0001 C CNN
 F 1 "GND" H 2605 2127 50  0000 C CNN
 F 2 "" H 2600 2300 50  0001 C CNN
@@
 Text GLabel 9650 2850 0    50   Output ~ 0
 PWM4
-Text GLabel 9550 4600 0    50   Input ~ 0
+Text GLabel 9550 4750 0    50   Input ~ 0
 PWM4
 Wire Wire Line
-	9550 4600 9900 4600
-$Comp
-L Connector:Conn_01x06_Male J?
-U 1 1 5FA8DBDA
-P 10100 4900
-AR Path="/5F475AB3/5FA8DBDA" Ref="J?"  Part="1"
-AR Path="/5F505E68/5FA8DBDA" Ref="J11"  Part="1"
-F 0 "J11" H 10072 4737 50  0000 R CNN
-F 1 "Conn_01x06_Male" H 10072 4828 50  0000 R CNN
-F 2 "Connector_Molex:Molex_CLIK-Mate_502443-0670_1x06-1MP_P2.00mm_Vertical" H 10100 4900 50  0001 C CNN
-F 3 "~" H 10100 4900 50  0001 C CNN
-F 4 "CLIC-Mate 502443-0670" H 10072 4919 50  0000 R CNN "Name"
-F 5 "Molex" H 10100 4900 50  0001 C CNN "Manufacturer"
-	1    10100 4900
-	-1   0    0    1
-$EndComp
+	9550 4750 9900 4750
 $Comp
 L Device:C C?
@@
 P 7350 2550
 AR Path="/5F4C6CE4/5FA9A4D8" Ref="C?"  Part="1"
-AR Path="/5F505E68/5FA9A4D8" Ref="C21"  Part="1"
-F 0 "C21" H 7465 2596 50  0000 L CNN
+AR Path="/5F505E68/5FA9A4D8" Ref="C23"  Part="1"
+F 0 "C23" H 7465 2596 50  0000 L CNN
 F 1 "100nF" H 7465 2505 50  0000 L CNN
 F 2 "" H 7388 2400 50  0001 C CNN
@@
 Text Notes 9400 1750 0    100  ~ 0
 Connectors
+$Comp
+L 74xx:74HC595 U?
+U 1 1 6023EEEB
+P 3450 3000
+AR Path="/5F4C6CE4/6023EEEB" Ref="U?"  Part="1"
+AR Path="/5F505E68/6023EEEB" Ref="U11"  Part="1"
+F 0 "U11" H 3450 3781 50  0000 C CNN
+F 1 "74HC595" H 3450 3690 50  0000 C CNN
+F 2 "MK2Library:SN74HC595PWR" H 3450 3000 50  0001 C CNN
+F 3 "http://www.ti.com/lit/ds/symlink/sn74hc595.pdf" H 3450 3000 50  0001 C CNN
+F 4 "SN74HC595PWR" H 3450 3000 50  0001 C CNN "Name"
+F 5 "Texas Instruments" H 3450 3000 50  0001 C CNN "Manufacturer"
+	1    3450 3000
+	1    0    0    -1
+$EndComp
+$Comp
+L Connector:Conn_01x06_Male J?
+U 1 1 60249757
+P 10100 4050
+AR Path="/5F475AB3/60249757" Ref="J?"  Part="1"
+AR Path="/5F4C6CE4/60249757" Ref="J?"  Part="1"
+AR Path="/5F505E68/60249757" Ref="J12"  Part="1"
+F 0 "J12" H 10072 3887 50  0000 R CNN
+F 1 "Conn_02x03_Male" H 10072 3978 50  0000 R CNN
+F 2 "MK2Library:901303206" H 10100 4050 50  0001 C CNN
+F 3 "~" H 10100 4050 50  0001 C CNN
+F 4 "90130-3206" H 10072 4069 50  0000 R CNN "Name"
+F 5 "Molex" H 10100 4050 50  0001 C CNN "Manufacturer"
+	1    10100 4050
+	-1   0    0    1
+$EndComp
+NoConn ~ 9900 3750
+$Comp
+L Connector:Conn_01x06_Male J?
+U 1 1 6022FE7E
+P 10100 5050
+AR Path="/5F475AB3/6022FE7E" Ref="J?"  Part="1"
+AR Path="/5F4C6CE4/6022FE7E" Ref="J?"  Part="1"
+AR Path="/5F505E68/6022FE7E" Ref="J13"  Part="1"
+F 0 "J13" H 10072 4887 50  0000 R CNN
+F 1 "Conn_02x03_Male" H 10072 4978 50  0000 R CNN
+F 2 "MK2Library:901303206" H 10100 5050 50  0001 C CNN
+F 3 "~" H 10100 5050 50  0001 C CNN
+F 4 "90130-3206" H 10072 5069 50  0000 R CNN "Name"
+F 5 "Molex" H 10100 5050 50  0001 C CNN "Manufacturer"
+	1    10100 5050
+	-1   0    0    1
+$EndComp
+$Comp
+L Connector:Conn_01x12_Male J11
+U 1 1 6024674F
+P 10100 2650
+AR Path="/5F505E68/6024674F" Ref="J11"  Part="1"
+AR Path="/5F4C637B/6024674F" Ref="J?"  Part="1"
+AR Path="/5F455032/6024674F" Ref="J?"  Part="1"
+F 0 "J11" H 10208 3421 50  0000 C CNN
+F 1 "Conn_02x6_Male" H 10208 3330 50  0000 C CNN
+F 2 "Connector_PinSocket_2.54mm:PinSocket_2x06_P2.54mm_Horizontal" H 10100 2650 50  0001 C CNN
+F 3 "~" H 10100 2650 50  0001 C CNN
+F 4 "T821112A1R100CEU" H 10208 3239 50  0000 C CNN "Name"
+F 5 "AMPHENOL ICC" H 10100 2650 50  0001 C CNN "Manufacturer"
+	1    10100 2650
+	-1   0    0    1
+$EndComp
+$Comp
+L power:PWR_FLAG #FLG?
+U 1 1 60304507
+P 9850 2950
+AR Path="/5F455032/60304507" Ref="#FLG?"  Part="1"
+AR Path="/5F4C637B/60304507" Ref="#FLG?"  Part="1"
+AR Path="/5F505E68/60304507" Ref="#FLG0108"  Part="1"
+F 0 "#FLG0108" H 9850 3025 50  0001 C CNN
+F 1 "PWR_FLAG" H 9850 3123 50  0000 C CNN
+F 2 "" H 9850 2950 50  0001 C CNN
+F 3 "~" H 9850 2950 50  0001 C CNN
+	1    9850 2950
+	1    0    0    -1
+$EndComp
+Connection ~ 9850 2950
+Wire Wire Line
+	9850 2950 9900 2950
+Text Label 3300 2000 2    50   ~ 0
+pwr12
 $EndSCHEMATC

Commit message: PCB design is updated
Parts:
- C22, C23: footprint (none) -> Capacitor_SMD:C_1206_3216Metric; Manufacturer (none) -> Kemet; Name (none) -> C1206C104K5RACTU
- J12, J13: value Conn_02x03_Male -> Conn_01x06_Male; footprint MK2Library:901303206 -> MK2Library:Molex_MicroClasp_55932-0610_1x06_P2.00mm_Vertical; Name 90130-3206 -> 55932-0610
Changed lines of the file:
@@
 Wire Wire Line
 	2900 2000 3450 2000
-Wire Wire Line
-	2400 2000 2600 2000
-$Comp
-L Device:C C?
-U 1 1 5F9DF246
-P 2600 2150
-AR Path="/5F4C6CE4/5F9DF246" Ref="C?"  Part="1"
-AR Path="/5F505E68/5F9DF246" Ref="C22"  Part="1"
-F 0 "C22" H 2715 2196 50  0000 L CNN
-F 1 "100nF" H 2715 2105 50  0000 L CNN
-F 2 "" H 2638 2000 50  0001 C CNN
-F 3 "~" H 2600 2150 50  0001 C CNN
-	1    2600 2150
-	1    0    0    -1
-$EndComp
-Connection ~ 2600 2000
-Wire Wire Line
-	2600 2000 2900 2000
 $Comp
 L power:GND #PWR?
@@
 Wire Wire Line
 	9550 4750 9900 4750
-$Comp
-L Device:C C?
-U 1 1 5FA9A4D8
-P 7350 2550
-AR Path="/5F4C6CE4/5FA9A4D8" Ref="C?"  Part="1"
-AR Path="/5F505E68/5FA9A4D8" Ref="C23"  Part="1"
-F 0 "C23" H 7465 2596 50  0000 L CNN
-F 1 "100nF" H 7465 2505 50  0000 L CNN
-F 2 "" H 7388 2400 50  0001 C CNN
-F 3 "~" H 7350 2550 50  0001 C CNN
-	1    7350 2550
-	1    0    0    -1
-$EndComp
 Text Notes 5900 1650 0    100  ~ 0
 Magnetic Encoder
@@
 AR Path="/5F505E68/60249757" Ref="J12"  Part="1"
 F 0 "J12" H 10072 3887 50  0000 R CNN
-F 1 "Conn_02x03_Male" H 10072 3978 50  0000 R CNN
-F 2 "MK2Library:901303206" H 10100 4050 50  0001 C CNN
+F 1 "Conn_01x06_Male" H 10072 3978 50  0000 R CNN
+F 2 "MK2Library:Molex_MicroClasp_55932-0610_1x06_P2.00mm_Vertical" H 10100 4050 50  0001 C CNN
 F 3 "~" H 10100 4050 50  0001 C CNN
-F 4 "90130-3206" H 10072 4069 50  0000 R CNN "Name"
+F 4 "55932-0610 " H 10072 4069 50  0000 R CNN "Name"
 F 5 "Molex" H 10100 4050 50  0001 C CNN "Manufacturer"
 	1    10100 4050
@@
 AR Path="/5F505E68/6022FE7E" Ref="J13"  Part="1"
 F 0 "J13" H 10072 4887 50  0000 R CNN
-F 1 "Conn_02x03_Male" H 10072 4978 50  0000 R CNN
-F 2 "MK2Library:901303206" H 10100 5050 50  0001 C CNN
+F 1 "Conn_01x06_Male" H 10072 4978 50  0000 R CNN
+F 2 "MK2Library:Molex_MicroClasp_55932-0610_1x06_P2.00mm_Vertical" H 10100 5050 50  0001 C CNN
 F 3 "~" H 10100 5050 50  0001 C CNN
-F 4 "90130-3206" H 10072 5069 50  0000 R CNN "Name"
+F 4 "55932-0610" H 10072 5069 50  0000 R CNN "Name"
 F 5 "Molex" H 10100 5050 50  0001 C CNN "Manufacturer"
 	1    10100 5050
@@
 Text Label 3300 2000 2    50   ~ 0
 pwr12
+$Comp
+L Device:C C?
+U 1 1 603335FB
+P 7350 2550
+AR Path="/5F4C6CE4/603335FB" Ref="C?"  Part="1"
+AR Path="/5F475AB3/603335FB" Ref="C?"  Part="1"
+AR Path="/5F505E68/603335FB" Ref="C23"  Part="1"
+F 0 "C23" H 7465 2596 50  0000 L CNN
+F 1 "100nF" H 7465 2505 50  0000 L CNN
+F 2 "Capacitor_SMD:C_1206_3216Metric" H 7388 2400 50  0001 C CNN
+F 3 "~" H 7350 2550 50  0001 C CNN
+F 4 "C1206C104K5RACTU" H 7350 2550 50  0001 C CNN "Name"
+F 5 "Kemet" H 7350 2550 50  0001 C CNN "Manufacturer"
+	1    7350 2550
+	1    0    0    -1
+$EndComp
+Wire Wire Line
+	2400 2000 2600 2000
+$Comp
+L Device:C C?
+U 1 1 6033F2EA
+P 2600 2150
+AR Path="/5F4C6CE4/6033F2EA" Ref="C?"  Part="1"
+AR Path="/5F475AB3/6033F2EA" Ref="C?"  Part="1"
+AR Path="/5F505E68/6033F2EA" Ref="C22"  Part="1"
+F 0 "C22" H 2715 2196 50  0000 L CNN
+F 1 "100nF" H 2715 2105 50  0000 L CNN
+F 2 "Capacitor_SMD:C_1206_3216Metric" H 2638 2000 50  0001 C CNN
+F 3 "~" H 2600 2150 50  0001 C CNN
+F 4 "C1206C104K5RACTU" H 2600 2150 50  0001 C CNN "Name"
+F 5 "Kemet" H 2600 2150 50  0001 C CNN "Manufacturer"
+	1    2600 2150
+	1    0    0    -1
+$EndComp
+Connection ~ 2600 2000
+Wire Wire Line
+	2600 2000 2900 2000
 $EndSCHEMATC

Commit message: all components are connected
Parts:
- J11: footprint Connector_PinSocket_2.54mm:PinSocket_2x06_P2.54mm_Horizontal -> Connector_IDC:IDC-Header_2x06_P2.54mm_Horizontal
Connections:
- net CLKEn4: now also J11.11 (Pin_11), J12.6 (Pin_6); no longer J11.5 (Pin_5), J12.3 (Pin_3)
- net GND: now also J11.3 (Pin_3), J12.2 (Pin_2); no longer J11.2 (Pin_2), J13.1 (Pin_1)
- net MISO4: now also J11.8 (Pin_8), J12.5 (Pin_5); no longer J11.6 (Pin_6), J12.4 (Pin_4)
- net PO-CLKDr4: now also J11.12 (Pin_12), J13.6 (Pin_6); no longer J11.11 (Pin_11), J13.4 (Pin_4)
- net PO-CLKEn4: now also J11.6 (Pin_6), J13.1 (Pin_1); no longer J11.8 (Pin_8), J12.1 (Pin_1)
- net PWM4: now also J11.9 (Pin_9), J13.5 (Pin_5); no longer J11.4 (Pin_4), J13.6 (Pin_6)
- net SH-CLKDr4: now also J11.7 (Pin_7), J13.4 (Pin_4); no longer J11.12 (Pin_12), J13.5 (Pin_5)
- net SH-CLKEn4: now also J11.4 (Pin_4), J13.2 (Pin_2); no longer J11.9 (Pin_9), J12.5 (Pin_5)
- net SerialDataDr4: now also J11.5 (Pin_5), J12.4 (Pin_4); no longer J11.10 (Pin_10), J13.3 (Pin_3)
- net SerialDataInEn4: now also J11.10 (Pin_10); no longer J11.7 (Pin_7)
- net SerialDataOutEn4: now also J13.3 (Pin_3); no longer J12.2 (Pin_2)
- net VCCF3v3: now also J11.2 (Pin_2); no longer J11.3 (Pin_3)
- net VMC: now also J12.1 (Pin_1); no longer J13.2 (Pin_2)
Changed lines of the file:
@@
 	9650 2050 9900 2050
 Wire Wire Line
+	9650 2550 9900 2550
+Wire Wire Line
+	9650 2250 9900 2250
+Wire Wire Line
+	9650 2350 9900 2350
+Wire Wire Line
+	9650 2450 9900 2450
+Wire Wire Line
+	9650 2850 9900 2850
+Wire Wire Line
+	9650 2650 9900 2650
+Wire Wire Line
+	9650 2750 9900 2750
+Wire Wire Line
 	9650 2150 9900 2150
-Wire Wire Line
-	9650 2250 9900 2250
-Wire Wire Line
-	9650 2350 9900 2350
-Wire Wire Line
-	9650 2450 9900 2450
-Wire Wire Line
-	9650 2550 9900 2550
-Wire Wire Line
-	9650 2650 9900 2650
-Wire Wire Line
-	9650 2750 9900 2750
-Wire Wire Line
-	9650 2850 9900 2850
-Wire Wire Line
-	9650 2950 9850 2950
-Text GLabel 9650 2750 0    50   Output ~ 0
+Text GLabel 9650 2150 0    50   Output ~ 0
 CLKEn4
+Text GLabel 9650 2450 0    50   Output ~ 0
+MISO4
+Text GLabel 9650 2850 0    50   Output ~ 0
+SH-CLKEn4
+Text GLabel 9650 2250 0    50   Output ~ 0
+SerialDataInEn4
 Text GLabel 9650 2650 0    50   Output ~ 0
-MISO4
-Text GLabel 9650 2350 0    50   Output ~ 0
-SH-CLKEn4
-Text GLabel 9650 2550 0    50   Output ~ 0
-SerialDataInEn4
-Text GLabel 9650 2450 0    50   Output ~ 0
 PO-CLKEn4
 $Comp
@@
 	1    0    0    -1
 $EndComp
-Text GLabel 9650 2150 0    50   Output ~ 0
+Text GLabel 9650 2050 0    50   Output ~ 0
 PO-CLKDr4
-Text GLabel 9650 2050 0    50   Output ~ 0
+Text GLabel 9650 2550 0    50   Output ~ 0
 SH-CLKDr4
-Text GLabel 9650 2950 0    50   Output ~ 0
+Text GLabel 9650 3050 0    50   Output ~ 0
 VCCF3v3
-Text GLabel 9650 2250 0    50   Output ~ 0
+Text GLabel 9650 2750 0    50   Output ~ 0
 SerialDataDr4
 Text GLabel 9650 3150 0    50   Output ~ 0
 VMC
 Wire Wire Line
-	9650 3050 9900 3050
+	9650 3050 9850 3050
 Wire Wire Line
 	9650 3150 9900 3150
 Wire Wire Line
+	9650 5150 9900 5150
+Wire Wire Line
 	9650 3850 9900 3850
 Wire Wire Line
-	9650 3950 9900 3950
-Wire Wire Line
-	9650 4050 9900 4050
-Wire Wire Line
-	9650 4150 9900 4150
-Wire Wire Line
-	9650 4250 9900 4250
-Text GLabel 9650 4050 0    50   Input ~ 0
+	9650 3750 9900 3750
+Wire Wire Line
+	9650 5050 9900 5050
+Wire Wire Line
+	9650 5250 9900 5250
+Text GLabel 9650 3750 0    50   Input ~ 0
 CLKEn4
-Text GLabel 9650 3950 0    50   Input ~ 0
+Text GLabel 9650 3850 0    50   Input ~ 0
 MISO4
-Text GLabel 9650 3850 0    50   Input ~ 0
+Text GLabel 9650 5150 0    50   Input ~ 0
 SH-CLKEn4
-Text GLabel 9650 4150 0    50   Input ~ 0
+Text GLabel 9650 5050 0    50   Input ~ 0
 SerialDataOutEn4
-Text GLabel 9650 4250 0    50   Input ~ 0
+Text GLabel 9650 5250 0    50   Input ~ 0
 PO-CLKEn4
-Text GLabel 9550 5050 0    50   Input ~ 0
+Text GLabel 9550 3950 0    50   Input ~ 0
 SerialDataDr4
-Text GLabel 9550 4850 0    50   Input ~ 0
+Text GLabel 9550 4950 0    50   Input ~ 0
 SH-CLKDr4
-Text GLabel 9550 4950 0    50   Input ~ 0
+Text GLabel 9550 4750 0    50   Input ~ 0
 PO-CLKDr4
-Text GLabel 9550 5150 0    50   Input ~ 0
+Text GLabel 9550 4250 0    50   Input ~ 0
 VMC
 Wire Wire Line
-	9550 4850 9900 4850
-Wire Wire Line
 	9550 4950 9900 4950
 Wire Wire Line
-	9550 5050 9900 5050
-Wire Wire Line
-	9550 5150 9900 5150
-Wire Wire Line
-	9900 5250 9150 5250
-Wire Wire Line
-	9150 5250 9150 5400
+	9550 4750 9900 4750
+Wire Wire Line
+	9550 3950 9900 3950
+Wire Wire Line
+	9550 4250 9900 4250
+Wire Wire Line
+	9900 4150 9150 4150
+Wire Wire Line
+	9150 4150 9150 4300
 $Comp
 L power:GND #PWR?
 U 1 1 5F53EADC
-P 9150 5400
+P 9150 4300
 AR Path="/5F4C6CE4/5F53EADC" Ref="#PWR?"  Part="1"
 AR Path="/5F4C6BF4/5F53EADC" Ref="#PWR?"  Part="1"
 AR Path="/5F505E68/5F53EADC" Ref="#PWR0134"  Part="1"
-F 0 "#PWR0134" H 9150 5150 50  0001 C CNN
-F 1 "GND" H 9155 5227 50  0000 C CNN
-F 2 "" H 9150 5400 50  0001 C CNN
-F 3 "" H 9150 5400 50  0001 C CNN
-	1    9150 5400
+F 0 "#PWR0134" H 9150 4050 50  0001 C CNN
+F 1 "GND" H 9155 4127 50  0000 C CNN
+F 2 "" H 9150 4300 50  0001 C CNN
+F 3 "" H 9150 4300 50  0001 C CNN
+	1    9150 4300
 	1    0    0    -1
 $EndComp
@@
 L power:GND #PWR?
 U 1 1 5F5DDE3D
-P 9650 3050
+P 9650 2950
 AR Path="/5F4C6CE4/5F5DDE3D" Ref="#PWR?"  Part="1"
 AR Path="/5F4C6BF4/5F5DDE3D" Ref="#PWR?"  Part="1"
 AR Path="/5F505E68/5F5DDE3D" Ref="#PWR0136"  Part="1"
-F 0 "#PWR0136" H 9650 2800 50  0001 C CNN
-F 1 "GND" H 9655 2877 50  0000 C CNN
-F 2 "" H 9650 3050 50  0001 C CNN
-F 3 "" H 9650 3050 50  0001 C CNN
-	1    9650 3050
+F 0 "#PWR0136" H 9650 2700 50  0001 C CNN
+F 1 "GND" H 9655 2777 50  0000 C CNN
+F 2 "" H 9650 2950 50  0001 C CNN
+F 3 "" H 9650 2950 50  0001 C CNN
+	1    9650 2950
 	0    1    1    0
 $EndComp
@@
 NoConn ~ 4100 3100
 NoConn ~ 4100 3200
-Text GLabel 9650 2850 0    50   Output ~ 0
+Text GLabel 9650 2350 0    50   Output ~ 0
 PWM4
-Text GLabel 9550 4750 0    50   Input ~ 0
+Text GLabel 9550 4850 0    50   Input ~ 0
 PWM4
 Wire Wire Line
-	9550 4750 9900 4750
+	9550 4850 9900 4850
 Text Notes 5900 1650 0    100  ~ 0
 Magnetic Encoder
@@
 	-1   0    0    1
 $EndComp
-NoConn ~ 9900 3750
 $Comp
 L Connector:Conn_01x06_Male J?
@@
 F 0 "J11" H 10208 3421 50  0000 C CNN
 F 1 "Conn_02x6_Male" H 10208 3330 50  0000 C CNN
-F 2 "Connector_PinSocket_2.54mm:PinSocket_2x06_P2.54mm_Horizontal" H 10100 2650 50  0001 C CNN
+F 2 "Connector_IDC:IDC-Header_2x06_P2.54mm_Horizontal" H 10100 2650 50  0001 C CNN
 F 3 "~" H 10100 2650 50  0001 C CNN
 F 4 "T821112A1R100CEU" H 10208 3239 50  0000 C CNN "Name"
@@
 L power:PWR_FLAG #FLG?
 U 1 1 60304507
-P 9850 2950
+P 9850 3050
 AR Path="/5F455032/60304507" Ref="#FLG?"  Part="1"
 AR Path="/5F4C637B/60304507" Ref="#FLG?"  Part="1"
 AR Path="/5F505E68/60304507" Ref="#FLG0108"  Part="1"
-F 0 "#FLG0108" H 9850 3025 50  0001 C CNN
-F 1 "PWR_FLAG" H 9850 3123 50  0000 C CNN
-F 2 "" H 9850 2950 50  0001 C CNN
-F 3 "~" H 9850 2950 50  0001 C CNN
-	1    9850 2950
-	1    0    0    -1
-$EndComp
-Connection ~ 9850 2950
-Wire Wire Line
-	9850 2950 9900 2950
+F 0 "#FLG0108" H 9850 3125 50  0001 C CNN
+F 1 "PWR_FLAG" H 9850 3223 50  0000 C CNN
+F 2 "" H 9850 3050 50  0001 C CNN
+F 3 "~" H 9850 3050 50  0001 C CNN
+	1    9850 3050
+	1    0    0    -1
+$EndComp
 Text Label 3300 2000 2    50   ~ 0
 pwr12
@@
 Wire Wire Line
 	2600 2000 2900 2000
+Connection ~ 9850 3050
+Wire Wire Line
+	9850 3050 9900 3050
+Wire Wire Line
+	9650 2950 9900 2950
+NoConn ~ 9900 4050
 $EndSCHEMATC
