File: mk2ee_kicad_project/supply.sch (KiCad schematic (older format))
At the start: 14 parts, among them J1 Conn_01x02, J2 Conn_01x12_Male, U1 NUCLEO-F411RE, U2 TSR_1-24150, U3 NCP718xSN330

Commit message: all components are checked
Parts:
- removed J1: Conn_01x02, MK2Library:Power, symbol Connector_Generic:Conn_01x02
- added J1: L712RA, MK2Library:Switchcraft-L712RA-0, symbol Switchcraft_-_L712RA:L712RA
- added TP4: TestPoint, TestPoint:TestPoint_Pad_D4.0mm, symbol Connector:TestPoint
- C1: footprint Capacitor_SMD:CP_Elec_6.3x5.8 -> Capacitor_SMD:CP_Elec_4x5.4; Manufacturer Kemet -> Panasonic; Name EDK106M063A9GAA -> EEEFK1E100R
- C2: footprint Capacitor_SMD:CP_Elec_6.3x5.8 -> Capacitor_SMD:CP_Elec_4x5.4
- C3, C4: Manufacturer (none) -> MULTICOMP PRO; Name (none) -> MC1206B102K500CT
- C5: Manufacturer Kemet -> Panasonic; Name EDK106M063A9GAA -> EEEFK1E101XP
- J2: value Conn_01x12_Male -> Conn_02x6_Male; footprint Connector_Molex:Molex_CLIK-Mate_502443-1270_1x12-1MP_P2.00mm_Vertical -> Connector_PinSocket_2.54mm:PinSocket_2x06_P2.54mm_Horizontal; Manufacturer Molex -> AMPHENOL ICC; Name CLIK-Mate 502443-1207 -> T821112A1R100CEU
- TP1, TP2, TP3: footprint (none) -> TestPoint:TestPoint_Pad_D4.0mm
- U2: Manufacturer (none) -> Traco Power; Name (none) -> TSR 1-2450
- U3: Manufacturer (none) -> ON SEMICONDUCTOR; Name (none) -> NCP718BSN330T1G
Connections:
- net +24V: no longer F1.P$1, TP1.1
- net +3V3: now also TP4.1
- net GND: now also J1.2 (SLEEVE)
- net MOSI1: now also U1.CN10_33 (PA10)
- net PWM1: now also U1.CN7_28 (PA0)
- new net pwr1: F1.P$1, J1.1 (CENTER_PIN), TP1.1
- no-connect marks 54 -> 53
Other:
- moved on the sheet: C1, C2, C3, C4, C5, F1, J2, TP1, TP2, TP3, U1A, U1B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

Commit message: all components are connected
Parts:
- J2: footprint Connector_PinSocket_2.54mm:PinSocket_2x06_P2.54mm_Horizontal -> Connector_IDC:IDC-Header_2x06_P2.54mm_Horizontal
- TP1, TP2, TP3, TP4: footprint TestPoint:TestPoint_Pad_D4.0mm -> TestPoint:TestPoint_Pad_D1.5mm
Connections:
- net +24V: now also J2.11 (Pin_11); no longer J2.1 (Pin_1)
- net +3V3: now also J2.12 (Pin_12); no longer J2.3 (Pin_3)
- net GND: now also J2.9 (Pin_9); no longer J2.2 (Pin_2)
- net PO-CLKDr1: now also J2.2 (Pin_2); no longer J2.11 (Pin_11)
- net PO-CLKEn1: now also U1.CN10_16 (PB12); no longer U1.CN10_24 (PB1)
- net PWM1: now also J2.3 (Pin_3); no longer J2.4 (Pin_4)
- net SH-CLKDr1: now also J2.5 (Pin_5); no longer J2.12 (Pin_12)
- net SH-CLKEn1: now also J2.10 (Pin_10), U1.CN10_30 (PB13); no longer J2.9 (Pin_9), U1.CN7_34 (PB0)
- net SerialDataOutDr1: now also J2.7 (Pin_7); no longer J2.10 (Pin_10)
- net SerialDataOutEn1: now also J2.4 (Pin_4); no longer J2.7 (Pin_7)
- net MOSI1: no longer names the net of U1.CN10_33 (PA10)
- net MOSI1: no longer J2.5 (Pin_5)
- new net CLK1: J2.1 (Pin_1), U1.CN7_34 (PB0)
Changed lines of the file:
@@
 Wire Wire Line
 	4300 5200 4650 5200
-Text GLabel 1350 6000 0    50   Output ~ 0
+Text GLabel 4200 6900 0    50   Output ~ 0
 SH-CLKEn1
-Text GLabel 4300 5900 0    50   Output ~ 0
+Text GLabel 4300 6800 0    50   Output ~ 0
 PO-CLKEn1
 Text GLabel 4300 5700 0    50   Input ~ 0
@@
 	4300 5700 4650 5700
 Wire Wire Line
-	4300 5900 4650 5900
-Wire Wire Line
-	1350 6000 1800 6000
+	4300 6800 4650 6800
+Wire Wire Line
+	4200 6900 4650 6900
 Text GLabel 1350 5400 0    50   Output ~ 0
 SerialDataOutEn1
@@
 NoConn ~ 4650 6600
 NoConn ~ 4650 6700
-NoConn ~ 4650 6800
-NoConn ~ 4650 6900
 NoConn ~ 4650 7000
 NoConn ~ 4650 7100
@@
 NoConn ~ 3400 5400
 Wire Wire Line
+	8850 4900 8600 4900
+Wire Wire Line
+	8850 5800 8600 5800
+Wire Wire Line
+	8850 4800 8600 4800
+Wire Wire Line
 	8850 5900 8600 5900
 Wire Wire Line
-	8850 5800 8600 5800
-Wire Wire Line
-	8850 5700 8600 5700
-Wire Wire Line
-	8850 5600 8600 5600
-Wire Wire Line
 	8850 5500 8600 5500
 Wire Wire Line
@@
 Wire Wire Line
 	8850 5000 8600 5000
-Text GLabel 8850 5200 2    50   Input ~ 0
-MOSI1
+Text GLabel 8850 4800 2    50   Input ~ 0
+CLK1
 Text GLabel 8850 5300 2    50   Output ~ 0
 MISO1
-Text GLabel 8850 5600 2    50   Input ~ 0
+Text GLabel 8850 5700 2    50   Input ~ 0
 SH-CLKEn1
-Text GLabel 8850 5400 2    50   Input ~ 0
+Text GLabel 8850 5100 2    50   Input ~ 0
 SerialDataOutEn1
 Text GLabel 8850 5500 2    50   Input ~ 0
 PO-CLKEn1
+Text GLabel 8850 4900 2    50   Input ~ 0
+PO-CLKDr1
+Text GLabel 8850 5200 2    50   Input ~ 0
+SH-CLKDr1
+Text GLabel 8850 5900 2    50   Input ~ 0
+VCCA3v3
+Text GLabel 8850 5400 2    50   Input ~ 0
+SerialDataOutDr1
 Text GLabel 8850 5800 2    50   Input ~ 0
-PO-CLKDr1
-Text GLabel 8850 5900 2    50   Input ~ 0
-SH-CLKDr1
-Text GLabel 8850 5000 2    50   Input ~ 0
-VCCA3v3
-Text GLabel 8850 5700 2    50   Input ~ 0
-SerialDataOutDr1
-Text GLabel 8850 4800 2    50   Input ~ 0
 VMA
 Wire Wire Line
-	8850 4800 8600 4800
-Wire Wire Line
-	9850 4900 9850 5050
-Wire Wire Line
-	8600 4900 9850 4900
+	8850 5700 8600 5700
+Wire Wire Line
+	9850 5600 9850 5750
+Wire Wire Line
+	8600 5600 9850 5600
 $Comp
 L power:GND #PWR?
 U 1 1 5FBF482F
-P 9850 5050
+P 9850 5750
 AR Path="/5F4C637B/5FBF482F" Ref="#PWR?"  Part="1"
 AR Path="/5F455032/5FBF482F" Ref="#PWR0102"  Part="1"
-F 0 "#PWR0102" H 9850 4800 50  0001 C CNN
-F 1 "GND" H 9855 4877 50  0000 C CNN
-F 2 "" H 9850 5050 50  0001 C CNN
-F 3 "" H 9850 5050 50  0001 C CNN
-	1    9850 5050
+F 0 "#PWR0102" H 9850 5500 50  0001 C CNN
+F 1 "GND" H 9855 5577 50  0000 C CNN
+F 2 "" H 9850 5750 50  0001 C CNN
+F 3 "" H 9850 5750 50  0001 C CNN
+	1    9850 5750
 	1    0    0    -1
 $EndComp
@@
 F 0 "J2" H 8508 6071 50  0000 C CNN
 F 1 "Conn_02x6_Male" H 8508 5980 50  0000 C CNN
-F 2 "Connector_PinSocket_2.54mm:PinSocket_2x06_P2.54mm_Horizontal" H 8400 5300 50  0001 C CNN
+F 2 "Connector_IDC:IDC-Header_2x06_P2.54mm_Horizontal" H 8400 5300 50  0001 C CNN
 F 3 "~" H 8400 5300 50  0001 C CNN
 F 4 "T821112A1R100CEU" H 8508 5889 50  0000 C CNN "Name"
@@
 Text GLabel 3850 4500 2    50   Input ~ 0
 VCCA5V
-Text GLabel 8850 5100 2    50   Input ~ 0
+Text GLabel 8850 5000 2    50   Input ~ 0
 PWM1
 NoConn ~ 4650 6500
@@
 F 0 "TP2" H 5158 1168 50  0000 L CNN
 F 1 "TestPoint" H 5158 1077 50  0001 L CNN
-F 2 "TestPoint:TestPoint_Pad_D4.0mm" H 5300 1050 50  0001 C CNN
+F 2 "TestPoint:TestPoint_Pad_D1.5mm" H 5300 1050 50  0001 C CNN
 F 3 "~" H 5300 1050 50  0001 C CNN
 	1    5100 1050
@@
 F 0 "TP1" H 4008 1168 50  0000 L CNN
 F 1 "TestPoint" H 4008 1077 50  0001 L CNN
-F 2 "TestPoint:TestPoint_Pad_D4.0mm" H 4150 1050 50  0001 C CNN
+F 2 "TestPoint:TestPoint_Pad_D1.5mm" H 4150 1050 50  0001 C CNN
 F 3 "~" H 4150 1050 50  0001 C CNN
 	1    3950 1050
@@
 F 0 "TP3" H 8258 1168 50  0000 L CNN
 F 1 "TestPoint" H 8258 1077 50  0001 L CNN
-F 2 "TestPoint:TestPoint_Pad_D4.0mm" H 8400 1050 50  0001 C CNN
+F 2 "TestPoint:TestPoint_Pad_D1.5mm" H 8400 1050 50  0001 C CNN
 F 3 "~" H 8400 1050 50  0001 C CNN
 	1    8200 1050
@@
 F 0 "TP4" H 7558 2618 50  0000 L CNN
 F 1 "TestPoint" H 7558 2527 50  0001 L CNN
-F 2 "TestPoint:TestPoint_Pad_D4.0mm" H 7700 2500 50  0001 C CNN
+F 2 "TestPoint:TestPoint_Pad_D1.5mm" H 7700 2500 50  0001 C CNN
 F 3 "~" H 7700 2500 50  0001 C CNN
 	1    7500 2500
@@
 Wire Wire Line
 	1350 5300 1800 5300
-Text GLabel 4300 5500 0    50   Output ~ 0
-MOSI1
-Wire Wire Line
-	4300 5500 4650 5500
 Text Label 7600 1300 2    50   ~ 0
 pwr3
 Text Label 7750 2750 2    50   ~ 0
 pwr4
+Wire Wire Line
+	1450 6000 1800 6000
+Text GLabel 1450 6000 0    50   Output ~ 0
+CLK1
+NoConn ~ 4650 5500
+NoConn ~ 4650 5900
 $EndSCHEMATC

Commit message: New 3D model of Base part and PCB design is fixed
Parts:
- added TP10: GND, TestPoint:TestPoint_THTPad_D1.0mm_Drill0.5mm, symbol Connector:TestPoint
- C3, C4: footprint Capacitor_SMD:C_1206_3216Metric -> Capacitor_SMD:C_1206_3216Metric_Pad1.42x1.75mm_HandSolder
- TP1, TP2, TP3, TP4: footprint TestPoint:TestPoint_Pad_D1.5mm -> TestPoint:TestPoint_THTPad_D1.0mm_Drill0.5mm
- U3: footprint Package_TO_SOT_SMD:SOT-23-5 -> Package_TO_SOT_SMD:SOT-23-5_HandSoldering
Connections:
- net +5V is gone; now on net +24V: C2.1, TP3.1, U1.CN7_6 (E5V), U2.3 (Vout)
- net +24V: no longer C1.1, F1.P$2, TP2.1, U2.1 (Vin)
- net GND: now also TP10.1
- new net pwr2: C1.1, F1.P$2, TP2.1, U2.1 (Vin)
Other:
- moved on the sheet: C3, C4, TP4, U3
Changed lines of the file:
@@
 L power:+3.3V #PWR0108
 U 1 1 5FBF4874
-P 7850 2550
+P 7850 2700
 AR Path="/5F455032/5FBF4874" Ref="#PWR0108"  Part="1"
 AR Path="/5F4C637B/5FBF4874" Ref="#PWR?"  Part="1"
-F 0 "#PWR0108" H 7850 2400 50  0001 C CNN
-F 1 "+3.3V" H 7865 2723 50  0000 C CNN
-F 2 "" H 7850 2550 50  0001 C CNN
-F 3 "" H 7850 2550 50  0001 C CNN
-	1    7850 2550
+F 0 "#PWR0108" H 7850 2550 50  0001 C CNN
+F 1 "+3.3V" H 7865 2873 50  0000 C CNN
+F 2 "" H 7850 2700 50  0001 C CNN
+F 3 "" H 7850 2700 50  0001 C CNN
+	1    7850 2700
 	1    0    0    -1
 $EndComp
@@
 F 0 "TP2" H 5158 1168 50  0000 L CNN
 F 1 "TestPoint" H 5158 1077 50  0001 L CNN
-F 2 "TestPoint:TestPoint_Pad_D1.5mm" H 5300 1050 50  0001 C CNN
+F 2 "TestPoint:TestPoint_THTPad_D1.0mm_Drill0.5mm" H 5300 1050 50  0001 C CNN
 F 3 "~" H 5300 1050 50  0001 C CNN
 	1    5100 1050
@@
 F 0 "TP1" H 4008 1168 50  0000 L CNN
 F 1 "TestPoint" H 4008 1077 50  0001 L CNN
-F 2 "TestPoint:TestPoint_Pad_D1.5mm" H 4150 1050 50  0001 C CNN
+F 2 "TestPoint:TestPoint_THTPad_D1.0mm_Drill0.5mm" H 4150 1050 50  0001 C CNN
 F 3 "~" H 4150 1050 50  0001 C CNN
 	1    3950 1050
@@
 L power:GND #PWR0121
 U 1 1 5FBF48E9
-P 6100 3400
+P 6100 3550
 AR Path="/5F455032/5FBF48E9" Ref="#PWR0121"  Part="1"
 AR Path="/5F475AB3/5FBF48E9" Ref="#PWR?"  Part="1"
 AR Path="/5F4C637B/5FBF48E9" Ref="#PWR?"  Part="1"
-F 0 "#PWR0121" H 6100 3150 50  0001 C CNN
-F 1 "GND" H 6105 3227 50  0000 C CNN
-F 2 "" H 6100 3400 50  0001 C CNN
-F 3 "" H 6100 3400 50  0001 C CNN
-	1    6100 3400
+F 0 "#PWR0121" H 6100 3300 50  0001 C CNN
+F 1 "GND" H 6105 3377 50  0000 C CNN
+F 2 "" H 6100 3550 50  0001 C CNN
+F 3 "" H 6100 3550 50  0001 C CNN
+	1    6100 3550
 	1    0    0    -1
 $EndComp
@@
 L power:GND #PWR0122
 U 1 1 5FBF48EF
-P 7000 3300
+P 7000 3450
 AR Path="/5F455032/5FBF48EF" Ref="#PWR0122"  Part="1"
 AR Path="/5F475AB3/5FBF48EF" Ref="#PWR?"  Part="1"
 AR Path="/5F4C637B/5FBF48EF" Ref="#PWR?"  Part="1"
-F 0 "#PWR0122" H 7000 3050 50  0001 C CNN
-F 1 "GND" H 7005 3127 50  0000 C CNN
-F 2 "" H 7000 3300 50  0001 C CNN
-F 3 "" H 7000 3300 50  0001 C CNN
-	1    7000 3300
+F 0 "#PWR0122" H 7000 3200 50  0001 C CNN
+F 1 "GND" H 7005 3277 50  0000 C CNN
+F 2 "" H 7000 3450 50  0001 C CNN
+F 3 "" H 7000 3450 50  0001 C CNN
+	1    7000 3450
 	1    0    0    -1
 $EndComp
@@
 L power:GND #PWR0123
 U 1 1 5FBF48F5
-P 7850 3400
+P 7850 3550
 AR Path="/5F455032/5FBF48F5" Ref="#PWR0123"  Part="1"
 AR Path="/5F475AB3/5FBF48F5" Ref="#PWR?"  Part="1"
 AR Path="/5F4C637B/5FBF48F5" Ref="#PWR?"  Part="1"
-F 0 "#PWR0123" H 7850 3150 50  0001 C CNN
-F 1 "GND" H 7855 3227 50  0000 C CNN
-F 2 "" H 7850 3400 50  0001 C CNN
-F 3 "" H 7850 3400 50  0001 C CNN
-	1    7850 3400
-	1    0    0    -1
-$EndComp
-Wire Wire Line
-	6100 2750 6100 2950
-Wire Wire Line
-	7850 2750 7850 2950
-Wire Wire Line
-	7850 3250 7850 3400
-Wire Wire Line
-	6100 3250 6100 3400
-Connection ~ 7850 2750
-Connection ~ 6100 2750
-Text GLabel 8150 2750 2    50   Output ~ 0
+F 0 "#PWR0123" H 7850 3300 50  0001 C CNN
+F 1 "GND" H 7855 3377 50  0000 C CNN
+F 2 "" H 7850 3550 50  0001 C CNN
+F 3 "" H 7850 3550 50  0001 C CNN
+	1    7850 3550
+	1    0    0    -1
+$EndComp
+Wire Wire Line
+	6100 2900 6100 3100
+Wire Wire Line
+	7850 2900 7850 3100
+Wire Wire Line
+	7850 3400 7850 3550
+Wire Wire Line
+	6100 3400 6100 3550
+Connection ~ 7850 2900
+Connection ~ 6100 2900
+Text GLabel 8150 2900 2    50   Output ~ 0
 VCCA3v3
 Wire Wire Line
-	7850 2750 8150 2750
+	7850 2900 8150 2900
 $Comp
 L Device:C C?
 U 1 1 5FBF4904
-P 6100 3100
+P 6100 3250
 AR Path="/5F475AB3/5FBF4904" Ref="C?"  Part="1"
 AR Path="/5F455032/5FBF4904" Ref="C3"  Part="1"
 AR Path="/5F4C637B/5FBF4904" Ref="C?"  Part="1"
-F 0 "C3" H 6215 3146 50  0000 L CNN
-F 1 "1uF" H 6215 3055 50  0000 L CNN
-F 2 "Capacitor_SMD:C_1206_3216Metric" H 6138 2950 50  0001 C CNN
-F 3 "~" H 6100 3100 50  0001 C CNN
-F 4 "MC1206B102K500CT" H 6100 3100 50  0001 C CNN "Name"
-F 5 "MULTICOMP PRO" H 6100 3100 50  0001 C CNN "Manufacturer"
-	1    6100 3100
+F 0 "C3" H 6215 3296 50  0000 L CNN
+F 1 "1uF" H 6215 3205 50  0000 L CNN
+F 2 "Capacitor_SMD:C_1206_3216Metric_Pad1.42x1.75mm_HandSolder" H 6138 3100 50  0001 C CNN
+F 3 "~" H 6100 3250 50  0001 C CNN
+F 4 "MC1206B102K500CT" H 6100 3250 50  0001 C CNN "Name"
+F 5 "MULTICOMP PRO" H 6100 3250 50  0001 C CNN "Manufacturer"
+	1    6100 3250
 	1    0    0    -1
 $EndComp
@@
 L Device:C C?
 U 1 1 5FBF490A
-P 7850 3100
+P 7850 3250
 AR Path="/5F475AB3/5FBF490A" Ref="C?"  Part="1"
 AR Path="/5F455032/5FBF490A" Ref="C4"  Part="1"
 AR Path="/5F4C637B/5FBF490A" Ref="C?"  Part="1"
-F 0 "C4" H 7965 3146 50  0000 L CNN
-F 1 "1uF" H 7965 3055 50  0000 L CNN
-F 2 "Capacitor_SMD:C_1206_3216Metric" H 7888 2950 50  0001 C CNN
-F 3 "~" H 7850 3100 50  0001 C CNN
-F 4 "MC1206B102K500CT" H 7850 3100 50  0001 C CNN "Name"
-F 5 "MULTICOMP PRO" H 7850 3100 50  0001 C CNN "Manufacturer"
-	1    7850 3100
+F 0 "C4" H 7965 3296 50  0000 L CNN
+F 1 "1uF" H 7965 3205 50  0000 L CNN
+F 2 "Capacitor_SMD:C_1206_3216Metric_Pad1.42x1.75mm_HandSolder" H 7888 3100 50  0001 C CNN
+F 3 "~" H 7850 3250 50  0001 C CNN
+F 4 "MC1206B102K500CT" H 7850 3250 50  0001 C CNN "Name"
+F 5 "MULTICOMP PRO" H 7850 3250 50  0001 C CNN "Manufacturer"
+	1    7850 3250
 	1    0    0    -1
 $EndComp
@@
 L Regulator_Linear:NCP718xSN330 U?
 U 1 1 5FBF4910
-P 7000 2850
+P 7000 3000
 AR Path="/5F475AB3/5FBF4910" Ref="U?"  Part="1"
 AR Path="/5F455032/5FBF4910" Ref="U3"  Part="1"
 AR Path="/5F4C637B/5FBF4910" Ref="U?"  Part="1"
-F 0 "U3" H 7000 3217 50  0000 C CNN
-F 1 "NCP718xSN330" H 7000 3126 50  0000 C CNN
-F 2 "Package_TO_SOT_SMD:SOT-23-5" H 7000 3200 50  0001 C CNN
-F 3 "https://www.onsemi.com/pub/Collateral/NCP718-D.PDF" H 7000 3350 50  0001 C CNN
-F 4 "NCP718BSN330T1G" H 7000 2850 50  0001 C CNN "Name"
-F 5 "ON SEMICONDUCTOR" H 7000 2850 50  0001 C CNN "Manufacturer"
-	1    7000 2850
-	1    0    0    -1
-$EndComp
-Wire Wire Line
-	7000 3150 7000 3300
-Wire Wire Line
-	6100 2750 6500 2750
-Wire Wire Line
-	6500 2750 6500 2850
-Wire Wire Line
-	6500 2850 6700 2850
-Connection ~ 6500 2750
-Wire Wire Line
-	6500 2750 6700 2750
-Wire Wire Line
-	5100 1300 5100 2750
-Wire Wire Line
-	5100 2750 6100 2750
+F 0 "U3" H 7000 3367 50  0000 C CNN
+F 1 "NCP718xSN330" H 7000 3276 50  0000 C CNN
+F 2 "Package_TO_SOT_SMD:SOT-23-5_HandSoldering" H 7000 3350 50  0001 C CNN
+F 3 "https://www.onsemi.com/pub/Collateral/NCP718-D.PDF" H 7000 3500 50  0001 C CNN
+F 4 "NCP718BSN330T1G" H 7000 3000 50  0001 C CNN "Name"
+F 5 "ON SEMICONDUCTOR" H 7000 3000 50  0001 C CNN "Manufacturer"
+	1    7000 3000
+	1    0    0    -1
+$EndComp
+Wire Wire Line
+	7000 3300 7000 3450
+Wire Wire Line
+	6100 2900 6500 2900
+Wire Wire Line
+	6500 2900 6500 3000
+Wire Wire Line
+	6500 3000 6700 3000
+Connection ~ 6500 2900
+Wire Wire Line
+	6500 2900 6700 2900
+Wire Wire Line
+	5100 2900 6100 2900
 $Comp
 L power:+24V #PWR0130
 U 1 1 5FC09960
-P 6100 2600
+P 6100 2750
 AR Path="/5F455032/5FC09960" Ref="#PWR0130"  Part="1"
 AR Path="/5F4C637B/5FC09960" Ref="#PWR?"  Part="1"
-F 0 "#PWR0130" H 6100 2450 50  0001 C CNN
-F 1 "+24V" H 6115 2773 50  0000 C CNN
-F 2 "" H 6100 2600 50  0001 C CNN
-F 3 "" H 6100 2600 50  0001 C CNN
-	1    6100 2600
+F 0 "#PWR0130" H 6100 2600 50  0001 C CNN
+F 1 "+24V" H 6115 2923 50  0000 C CNN
+F 2 "" H 6100 2750 50  0001 C CNN
+F 3 "" H 6100 2750 50  0001 C CNN
+	1    6100 2750
 	1    0    0    -1
 $EndComp
@@
 F 0 "TP3" H 8258 1168 50  0000 L CNN
 F 1 "TestPoint" H 8258 1077 50  0001 L CNN
-F 2 "TestPoint:TestPoint_Pad_D1.5mm" H 8400 1050 50  0001 C CNN
+F 2 "TestPoint:TestPoint_THTPad_D1.0mm_Drill0.5mm" H 8400 1050 50  0001 C CNN
 F 3 "~" H 8400 1050 50  0001 C CNN
 	1    8200 1050
@@
 $EndComp
 Wire Wire Line
-	7850 2550 7850 2750
-Wire Wire Line
-	6100 2600 6100 2750
+	7850 2700 7850 2900
+Wire Wire Line
+	6100 2750 6100 2900
 Text Notes 2150 950  0    100  ~ 0
 Input\nConnector
@@
 L Connector:TestPoint TP4
 U 1 1 6024378E
-P 7500 2500
+P 7500 2650
 AR Path="/5F455032/6024378E" Ref="TP4"  Part="1"
 AR Path="/5F4C637B/6024378E" Ref="TP?"  Part="1"
-F 0 "TP4" H 7558 2618 50  0000 L CNN
-F 1 "TestPoint" H 7558 2527 50  0001 L CNN
-F 2 "TestPoint:TestPoint_Pad_D1.5mm" H 7700 2500 50  0001 C CNN
-F 3 "~" H 7700 2500 50  0001 C CNN
-	1    7500 2500
-	1    0    0    -1
-$EndComp
-Wire Wire Line
-	7500 2750 7500 2500
-Wire Wire Line
-	7300 2750 7500 2750
-Connection ~ 7500 2750
-Wire Wire Line
-	7500 2750 7850 2750
+F 0 "TP4" H 7558 2768 50  0000 L CNN
+F 1 "TestPoint" H 7558 2677 50  0001 L CNN
+F 2 "TestPoint:TestPoint_THTPad_D1.0mm_Drill0.5mm" H 7700 2650 50  0001 C CNN
+F 3 "~" H 7700 2650 50  0001 C CNN
+	1    7500 2650
+	1    0    0    -1
+$EndComp
+Wire Wire Line
+	7500 2900 7500 2650
+Wire Wire Line
+	7300 2900 7500 2900
+Connection ~ 7500 2900
+Wire Wire Line
+	7500 2900 7850 2900
 Wire Wire Line
 	3000 1300 3550 1300
@@
 Text Label 7600 1300 2    50   ~ 0
 pwr3
-Text Label 7750 2750 2    50   ~ 0
+Text Label 7750 2900 2    50   ~ 0
 pwr4
 Wire Wire Line
@@
 NoConn ~ 4650 5500
 NoConn ~ 4650 5900
+Wire Wire Line
+	8200 1300 8200 2400
+Wire Wire Line
+	8200 2400 5100 2400
+Wire Wire Line
+	5100 2400 5100 2900
+$Comp
+L Connector:TestPoint TP10
+U 1 1 608AF637
+P 1650 2850
+AR Path="/5F455032/608AF637" Ref="TP10"  Part="1"
+AR Path="/5F4C637B/608AF637" Ref="TP?"  Part="1"
+F 0 "TP10" H 1708 2968 50  0000 L CNN
+F 1 "GND" H 1708 2877 50  0000 L CNN
+F 2 "TestPoint:TestPoint_THTPad_D1.0mm_Drill0.5mm" H 1850 2850 50  0001 C CNN
+F 3 "~" H 1850 2850 50  0001 C CNN
+	1    1650 2850
+	1    0    0    -1
+$EndComp
+$Comp
+L power:GND #PWR0104
+U 1 1 608AFE03
+P 1650 2850
+AR Path="/5F455032/608AFE03" Ref="#PWR0104"  Part="1"
+AR Path="/5F4C637B/608AFE03" Ref="#PWR?"  Part="1"
+F 0 "#PWR0104" H 1650 2600 50  0001 C CNN
+F 1 "GND" H 1655 2677 50  0000 C CNN
+F 2 "" H 1650 2850 50  0001 C CNN
+F 3 "" H 1650 2850 50  0001 C CNN
+	1    1650 2850
+	1    0    0    -1
+$EndComp
 $EndSCHEMATC
