File: mk2ee_kicad_project/MK2EE.kicad_pcb (KiCad board)
At the start: 2 copper layers, 179.9 x 168.9 mm, 99 parts, among them J1 L712RA, J10 Conn_01x02_Male, J11 Conn_02x6_Male, J12 Conn_01x06_Male, J13 Conn_01x06_Male, J2 Conn_02x6_Male, J3 Conn_01x02_Male, J4 Conn_02x03_Male, J5 Conn_02x03_Male, J6 Conn_01x04_Male, J7 Conn_01x04_Male, J8 Conn_02x03_Male, J9 Conn_02x03_Male, U1 NUCLEO-F411RE, U10 AS5047D-ATSM, U11 74HC595, U2 TSR_1-24150, U3 NCP718xSN330, U4 TSR_1-2465, U5 NCP718xSN330, U6 74HC595, U7 DRV8818PWP, U8 AS5047D-ATSM, U9 74HC595

Commit message: Thermal pad from stepper driver is modified
Parts:
- added C10: 0.22uF, Capacitor_SMD:C_1206_3216Metric_Pad1.42x1.75mm_HandSolder, B.Cu at (259.9, 93.2)
- added C11: 100nF, Capacitor_SMD:C_1206_3216Metric_Pad1.42x1.75mm_HandSolder, F.Cu at (252.3, 104.5)
- added C12: 100nF, Capacitor_SMD:C_1206_3216Metric_Pad1.42x1.75mm_HandSolder, B.Cu at (250.6, 91.1)
- added C13: 100nF, Capacitor_SMD:C_1206_3216Metric_Pad1.42x1.75mm_HandSolder, B.Cu at (240.0, 103.8)
- added C14: 100uF, Capacitor_SMD:CP_Elec_6.3x7.7, F.Cu at (263.1, 73.0)
- added C15: 1uF, Capacitor_SMD:C_1206_3216Metric_Pad1.42x1.75mm_HandSolder, F.Cu at (244.4, 73.7)
- added C16: 1uF, Capacitor_SMD:C_1206_3216Metric_Pad1.42x1.75mm_HandSolder, F.Cu at (253.6, 77.1)
- added C17: 10uF, Capacitor_SMD:CP_Elec_4x5.4, F.Cu at (231.8, 107.6)
- added C18: 10uF, Capacitor_SMD:CP_Elec_4x5.4, F.Cu at (239.4, 107.6)
- added C19: 100nF, Capacitor_SMD:C_1206_3216Metric_Pad1.42x1.75mm_HandSolder, B.Cu at (249.2, 82.7)
- added C20: 100nF, Capacitor_SMD:C_1206_3216Metric_Pad1.42x1.75mm_HandSolder, F.Cu at (246.8, 169.5)
- added C21: 100nF, Capacitor_SMD:C_1206_3216Metric_Pad1.42x1.75mm_HandSolder, F.Cu at (245.4, 154.4)
- added C6: 1000pF, Capacitor_SMD:C_1206_3216Metric_Pad1.42x1.75mm_HandSolder, B.Cu at (237.8, 101.2)
- added C7: 1000pF, Capacitor_SMD:C_1206_3216Metric_Pad1.42x1.75mm_HandSolder, B.Cu at (237.4, 96.5)
- added C8: 0.22uF, Capacitor_SMD:C_1206_3216Metric_Pad1.42x1.75mm_HandSolder, B.Cu at (259.4, 100.7)
- added C9: 0.22uF, Capacitor_SMD:C_1206_3216Metric_Pad1.42x1.75mm_HandSolder, B.Cu at (260.7, 97.1)
- added F2: Polyfuse, MK2Library:MINISMDC110, F.Cu at (235.3, 101.0)
- added F3: Polyfuse, MK2Library:MINISMDC110, F.Cu at (253.2, 71.1)
- added H5: MountingHole_3.2mm_M3, MountingHole:MountingHole_3.2mm_M3, F.Cu at (233.0, 73.0)
- added H5: MountingHole_3.2mm_M3, MountingHole:MountingHole_3.2mm_M3, F.Cu at (264.0, 104.0)
- added J10: Conn_01x02_Male, MK2Library:Molex_MicroClasp_55932-0210_1x02_P2.00mm_Vertical, B.Cu at (252.2, 188.2)
- added J3: Conn_01x02_Male, MK2Library:Molex_MicroClasp_55932-0210_1x02_P2.00mm_Vertical, F.Cu at (260.9, 125.0)
- added J4: Conn_02x03_Male, Connector_IDC:IDC-Header_2x03_P2.54mm_Horizontal, F.Cu at (267.3, 86.0)
- added J5: Conn_02x03_Male, Connector_IDC:IDC-Header_2x03_P2.54mm_Horizontal, F.Cu at (230.0, 91.0)
- added J6: Conn_01x04_Male, MK2Library:Molex_MicroClasp_55935-0430_1x04_P2.00mm_Horizontal, F.Cu at (232.0, 124.4)
- added J7: Conn_01x04_Male, MK2Library:Molex_MicroClasp_55935-0430_1x04_P2.00mm_Horizontal, B.Cu at (251.5, 118.5)
- added J8: Conn_02x03_Male, Connector_IDC:IDC-Header_2x03_P2.54mm_Horizontal, B.Cu at (268.1, 189.6)
- added J9: Conn_02x03_Male, Connector_IDC:IDC-Header_2x03_P2.54mm_Horizontal, B.Cu at (234.2, 184.5)
- added LED1: ASMB-KTF0-0A306, MK2Library:ASMBKTF00A306, F.Cu at (236.8, 153.9)
- added LED2: ASMB-KTF0-0A306, MK2Library:ASMBKTF00A306, F.Cu at (265.0, 153.9)
- added R1: 47k, Resistor_SMD:R_1206_3216Metric_Pad1.42x1.75mm_HandSolder, B.Cu at (232.8, 101.2)
- added R10: 100R, Resistor_SMD:R_1206_3216Metric_Pad1.42x1.75mm_HandSolder, F.Cu at (240.5, 158.2)
- added R11: 270R, Resistor_SMD:R_1206_3216Metric_Pad1.42x1.75mm_HandSolder, F.Cu at (233.1, 158.2)
- added R12: 82R, Resistor_SMD:R_1206_3216Metric_Pad1.42x1.75mm_HandSolder, F.Cu at (265.0, 158.2)
- added R13: 100R, Resistor_SMD:R_1206_3216Metric_Pad1.42x1.75mm_HandSolder, F.Cu at (268.7, 158.2)
- added R14: 270R, Resistor_SMD:R_1206_3216Metric_Pad1.42x1.75mm_HandSolder, F.Cu at (261.3, 158.2)
- added R2: 10k, Resistor_SMD:R_1206_3216Metric_Pad1.42x1.75mm_HandSolder, B.Cu at (240.0, 108.5)
- added R3: 10k, Resistor_SMD:R_1206_3216Metric_Pad1.42x1.75mm_HandSolder, B.Cu at (240.0, 106.1)
- added R4: 10k, Resistor_SMD:R_1206_3216Metric_Pad1.42x1.75mm_HandSolder, B.Cu at (227.3, 96.7)
- added R5: 10k, Resistor_SMD:R_1206_3216Metric_Pad1.42x1.75mm_HandSolder, B.Cu at (227.3, 99.1)
- added R6: 47k, Resistor_SMD:R_1206_3216Metric_Pad1.42x1.75mm_HandSolder, B.Cu at (232.5, 96.5)
- added R7: 0.43R, Resistor_SMD:R_1206_3216Metric_Pad1.42x1.75mm_HandSolder, B.Cu at (246.7, 105.9)
- added R8: 0.43R, Resistor_SMD:R_1206_3216Metric_Pad1.42x1.75mm_HandSolder, B.Cu at (243.4, 92.1)
- added R9: 82R, Resistor_SMD:R_1206_3216Metric_Pad1.42x1.75mm_HandSolder, F.Cu at (236.8, 158.2)
- added REF**: MountingHole_3.2mm_M3, MountingHole:MountingHole_3.2mm_M3, F.Cu at (251.2, 195.6)
- added REF**: MountingHole_3.2mm_M3, MountingHole:MountingHole_3.2mm_M3, F.Cu at (251.2, 174.6)
- added TP11: TestPoint, TestPoint:TestPoint_THTPad_D1.0mm_Drill0.5mm, F.Cu at (262.8, 115.8)
- added TP12: TestPoint, TestPoint:TestPoint_THTPad_D1.0mm_Drill0.5mm, F.Cu at (233.9, 173.8)
- added TP5: TestPoint, TestPoint:TestPoint_THTPad_D1.0mm_Drill0.5mm, F.Cu at (230.1, 112.8)
- added TP7: TestPoint, TestPoint:TestPoint_THTPad_D1.0mm_Drill0.5mm, F.Cu at (241.1, 112.1)
- added TP8: TestPoint, TestPoint:TestPoint_THTPad_D1.0mm_Drill0.5mm, F.Cu at (246.8, 70.8)
- added TP9: TestPoint, TestPoint:TestPoint_THTPad_D1.0mm_Drill0.5mm, F.Cu at (260.5, 80.6)
- added U4: TSR_1-2465, Converter_DCDC:Converter_DCDC_TRACO_TSR-1_THT, B.Cu at (232.7, 116.4)
- added U5: NCP718xSN330, Package_TO_SOT_SMD:SOT-23-5_HandSoldering, F.Cu at (247.2, 76.9)
- added U6: 74HC595, MK2Library:SN74HC595PWR, F.Cu at (249.1, 86.2)
- added U7: DRV8818PWR, MK2Library:DRV8818PWP, B.Cu at (249.2, 98.4)
- added U8: AS5047D-ATSM, MK2Library:AS5047D-ATSM, F.Cu at (251.2, 156.6)
- added U9: 74HC595, MK2Library:SN74HC595PWR, F.Cu at (251.2, 165.3)
- added mouse-bite-3mm-slot: VAL**, MK2Library:mouse-bite-3mm-slot, F.Cu at (251.1, 146.6)
- added mouse-bite-3mm-slot: VAL**, MK2Library:mouse-bite-3mm-slot, F.Cu at (248.5, 130.5)
- added mouse-bite-3mm-slot: VAL**, MK2Library:mouse-bite-3mm-slot, F.Cu at (215.3, 87.3)
- added mouse-bite-3mm-slot: VAL**, MK2Library:mouse-bite-3mm-slot, F.Cu at (219.6, 186.9)
- U7: value DRV8818PWP -> DRV8818PWR
Connections:
- U7 pad 29: (no net) -> GND
Routing:
- net VMB: track 177.0 -> 353.9 mm, vias 4 -> 8
- net GND: track 172.9 -> 281.0 mm, vias 28 -> 44
- net MISO3: track 107.5 -> 215.0 mm, vias 1 -> 2
- net PWM2: track 103.1 -> 206.1 mm, vias 2 -> 4
- net CLKEn3: track 97.3 -> 194.5 mm, vias 1 -> 2
- net PO-CLKEn3: track 61.0 -> 122.0 mm
- net SH-CLKEn3: track 59.0 -> 118.0 mm
- net SH-CLKDr2: track 47.2 -> 94.4 mm
- net PO-CLKDr2: track 45.5 -> 91.0 mm
- net /driver-1/2B: track 41.6 -> 83.2 mm, vias 1 -> 2
- net /driver-1/2A: track 39.9 -> 79.8 mm, vias 1 -> 2
- net SerialDataOutEn3: track 34.3 -> 68.5 mm, vias 1 -> 2
- net SerialDataInEn3: track 32.8 -> 65.7 mm
- net DIR: track 30.6 -> 61.2 mm, vias 3 -> 6
- net /driver-1/1B: track 29.3 -> 58.5 mm
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Other:
- board size 179.9 x 168.9 mm -> 243.9 x 168.9 mm
